File: DaughterBoard/untitled.kicad_sch (KiCad schematic)
At the start: 75 parts

Commit message: modhy commit
Parts:
- C10: renamed from C19; footprint GCM188R71C474KA55D:G-188_MUR-L -> Capacitor_SMD:C_0201_0603Metric
- C11: renamed from C17; footprint GCM188R71C474KA55D:G-188_MUR-L -> Capacitor_SMD:C_0201_0603Metric
- C12: renamed from C15; footprint GCM188R71C474KA55D:G-188_MUR-L -> Capacitor_SMD:C_0201_0603Metric
- C13: footprint GCM188R71C474KA55D:G-188_MUR-L -> Capacitor_SMD:C_0201_0603Metric
- C14: renamed from C11; footprint GCM188R71C474KA55D:G-188_MUR-L -> Capacitor_SMD:C_0201_0603Metric
- C15: renamed from C9; footprint GCM188R71C474KA55D:G-188_MUR-L -> Capacitor_SMD:C_0201_0603Metric
- C16: renamed from C7; footprint GCM188R71C474KA55D:G-188_MUR-L -> Capacitor_SMD:C_0201_0603Metric
- C17: renamed from C5; footprint GCM188R71C474KA55D:G-188_MUR-L -> Capacitor_SMD:C_0201_0603Metric
- C18: renamed from C3; footprint GCM188R71C474KA55D:G-188_MUR-L -> Capacitor_SMD:C_0201_0603Metric
- C19: renamed from C1; footprint GCM188R71C474KA55D:G-188_MUR-L -> Capacitor_SMD:C_0201_0603Metric
- C20: renamed from C22; footprint GCM188R71C474KA55D:G-188_MUR-L -> Capacitor_SMD:C_0201_0603Metric
- C21: renamed from C20; footprint GCM188R71C474KA55D:G-188_MUR-L -> Capacitor_SMD:C_0201_0603Metric
- C22: renamed from C18; footprint GCM188R71C474KA55D:G-188_MUR-L -> Capacitor_SMD:C_0201_0603Metric
- C23: renamed from C16; footprint GCM188R71C474KA55D:G-188_MUR-L -> Capacitor_SMD:C_0201_0603Metric
- C24: renamed from C14; footprint GCM188R71C474KA55D:G-188_MUR-L -> Capacitor_SMD:C_0201_0603Metric
- C25: renamed from C12; footprint GCM188R71C474KA55D:G-188_MUR-L -> Capacitor_SMD:C_0201_0603Metric
- C26: renamed from C10; footprint GCM188R71C474KA55D:G-188_MUR-L -> Capacitor_SMD:C_0201_0603Metric
- C27: renamed from C8; footprint GCM188R71C474KA55D:G-188_MUR-L -> Capacitor_SMD:C_0201_0603Metric
- C28: renamed from C6; footprint GCM188R71C474KA55D:G-188_MUR-L -> Capacitor_SMD:C_0201_0603Metric
- C29: renamed from C4; footprint GCM188R71C474KA55D:G-188_MUR-L -> Capacitor_SMD:C_0201_0603Metric
- C30: renamed from C2; footprint GCM188R71C474KA55D:G-188_MUR-L -> Capacitor_SMD:C_0201_0603Metric
- C31: renamed from C29; footprint GCM188R71C474KA55D:G-188_MUR-L -> Capacitor_SMD:C_0201_0603Metric
- C32: renamed from C27; footprint GCM188R71C474KA55D:G-188_MUR-L -> Capacitor_SMD:C_0201_0603Metric
- C33: renamed from C25; footprint GCM188R71C474KA55D:G-188_MUR-L -> Capacitor_SMD:C_0201_0603Metric
- C34: renamed from C23; footprint GCM188R71C474KA55D:G-188_MUR-L -> Capacitor_SMD:C_0603_1608Metric
- C35: renamed from C30; footprint GCM188R71C474KA55D:G-188_MUR-L -> Capacitor_SMD:C_0201_0603Metric
- C36: renamed from C28; footprint GCM188R71C474KA55D:G-188_MUR-L -> Capacitor_SMD:C_0201_0603Metric
- C37: renamed from C26; footprint GCM188R71C474KA55D:G-188_MUR-L -> Capacitor_SMD:C_0201_0603Metric
- C38: renamed from C24; footprint GCM188R71C474KA55D:G-188_MUR-L -> Capacitor_SMD:C_0201_0603Metric
- C9: renamed from C21; footprint GCM188R71C474KA55D:G-188_MUR-L -> Capacitor_SMD:C_0201_0603Metric
- R10: renamed from R5; value 10 Ohm -> 7.5 Ohm; footprint CRCW121010R0FKEAHP:RC1210N_VIS-L -> Resistor_SMD:R_1206_3216Metric
- R11: renamed from R3; value 10 Ohm -> 7.5 Ohm; footprint CRCW121010R0FKEAHP:RC1210N_VIS-L -> Resistor_SMD:R_1206_3216Metric
- R12: renamed from R1; value 10 Ohm -> 7.5 Ohm; footprint CRCW121010R0FKEAHP:RC1210N_VIS-L -> Resistor_SMD:R_1206_3216Metric
- R13: renamed from R22; footprint ERA-3AEB101V:RC0603N_PAN-L -> Resistor_SMD:R_0201_0603Metric
- R14: renamed from R20; footprint ERA-3AEB101V:RC0603N_PAN-L -> Resistor_SMD:R_0201_0603Metric
- R15: renamed from R18; footprint ERA-3AEB101V:RC0603N_PAN-L -> Resistor_SMD:R_0201_0603Metric
- R16: footprint ERA-3AEB101V:RC0603N_PAN-L -> Resistor_SMD:R_0201_0603Metric
- R17: renamed from R14; footprint ERA-3AEB101V:RC0603N_PAN-L -> Resistor_SMD:R_0201_0603Metric
- R18: renamed from R12; footprint ERA-3AEB101V:RC0603N_PAN-L -> Resistor_SMD:R_0201_0603Metric
- R19: renamed from R10; footprint ERA-3AEB101V:RC0603N_PAN-L -> Resistor_SMD:R_0201_0603Metric
- R2: renamed from R21; value 10 Ohm -> 7.5 Ohm; footprint CRCW121010R0FKEAHP:RC1210N_VIS-L -> Resistor_SMD:R_1206_3216Metric
- R20: renamed from R8; footprint ERA-3AEB101V:RC0603N_PAN-L -> Resistor_SMD:R_0201_0603Metric
- R21: renamed from R6; footprint ERA-3AEB101V:RC0603N_PAN-L -> Resistor_SMD:R_0201_0603Metric
- R22: renamed from R4; footprint ERA-3AEB101V:RC0603N_PAN-L -> Resistor_SMD:R_0201_0603Metric
- R23: renamed from R2; footprint ERA-3AEB101V:RC0603N_PAN-L -> Resistor_SMD:R_0201_0603Metric
- R24: renamed from R29; value 10 Ohm -> 7.5 Ohm; footprint CRCW121010R0FKEAHP:RC1210N_VIS-L -> Resistor_SMD:R_1206_3216Metric
- R25: renamed from R27; value 10 Ohm -> 7.5 Ohm; footprint CRCW121010R0FKEAHP:RC1210N_VIS-L -> Resistor_SMD:R_1206_3216Metric
- R26: renamed from R25; value 10 Ohm -> 7.5 Ohm; footprint CRCW121010R0FKEAHP:RC1210N_VIS-L -> Resistor_SMD:R_1206_3216Metric
- R27: renamed from R23; value 10 Ohm -> 7.5 Ohm; footprint CRCW121010R0FKEAHP:RC1210N_VIS-L -> Resistor_SMD:R_1206_3216Metric
- R28: renamed from R30; footprint ERA-3AEB101V:RC0603N_PAN-L -> Resistor_SMD:R_0201_0603Metric
- R29: renamed from R28; footprint ERA-3AEB101V:RC0603N_PAN-L -> Resistor_SMD:R_0201_0603Metric
- R3: renamed from R19; value 10 Ohm -> 7.5 Ohm; footprint CRCW121010R0FKEAHP:RC1210N_VIS-L -> Resistor_SMD:R_1206_3216Metric
- R30: renamed from R26; footprint ERA-3AEB101V:RC0603N_PAN-L -> Resistor_SMD:R_0201_0603Metric
- R31: renamed from R24; footprint ERA-3AEB101V:RC0603N_PAN-L -> Resistor_SMD:R_0201_0603Metric
- R4: renamed from R17; value 10 Ohm -> 7.5 Ohm; footprint CRCW121010R0FKEAHP:RC1210N_VIS-L -> Resistor_SMD:R_1206_3216Metric
- R5: renamed from R15; value 10 Ohm -> 7.5 Ohm; footprint CRCW121010R0FKEAHP:RC1210N_VIS-L -> Resistor_SMD:R_1206_3216Metric
- R6: renamed from R13; value 10 Ohm -> 7.5 Ohm; footprint CRCW121010R0FKEAHP:RC1210N_VIS-L -> Resistor_SMD:R_1206_3216Metric
- R7: renamed from R11; value 10 Ohm -> 7.5 Ohm
- R8: renamed from R9; value 10 Ohm -> 7.5 Ohm; footprint CRCW121010R0FKEAHP:RC1210N_VIS-L -> Resistor_SMD:R_1206_3216Metric
- TP18: renamed from TP11; footprint (none) -> TestPoint:TestPoint_Keystone_5010-5014_Multipurpose
- TP19: renamed from TP10; footprint (none) -> TestPoint:TestPoint_Keystone_5010-5014_Multipurpose
- TP20: renamed from TP9; footprint (none) -> TestPoint:TestPoint_Keystone_5010-5014_Multipurpose
- TP22: renamed from TP7; footprint (none) -> TestPoint:TestPoint_Keystone_5010-5014_Multipurpose
- TP23: renamed from TP6; footprint (none) -> TestPoint:TestPoint_Keystone_5010-5014_Multipurpose
- TP24: renamed from TP5; footprint (none) -> TestPoint:TestPoint_Keystone_5010-5014_Multipurpose
- TP25: renamed from TP4; footprint (none) -> TestPoint:TestPoint_Keystone_5010-5014_Multipurpose
- TP26: renamed from TP3; footprint (none) -> TestPoint:TestPoint_Keystone_5010-5014_Multipurpose
- TP27: renamed from TP2; footprint (none) -> TestPoint:TestPoint_Keystone_5010-5014_Multipurpose
- TP28: renamed from TP1; footprint (none) -> TestPoint:TestPoint_Keystone_5010-5014_Multipurpose
- TP29: renamed from TP15; footprint (none) -> TestPoint:TestPoint_Keystone_5010-5014_Multipurpose
- TP30: renamed from TP14; footprint (none) -> TestPoint:TestPoint_Keystone_5010-5014_Multipurpose
- TP31: renamed from TP13; footprint (none) -> TestPoint:TestPoint_Keystone_5010-5014_Multipurpose
- TP32: renamed from TP12; footprint (none) -> TestPoint:TestPoint_Keystone_5010-5014_Multipurpose
- renumbered R7 to R9, TP8 to TP21

Commit message: 90% DOBO is done
Parts:
- removed R10, R11, R12, R2, R24, R25, R26, R27, R3, R4, R5, R6, R8: 7.5 Ohm, Resistor_SMD:R_1206_3216Metric, symbol 2024-10-08_02-17-57:CRCW121010R0FKEAHP
- removed R7: 7.5 Ohm, CRCW121010R0FKEAHP:RC1210N_VIS-L, symbol 2024-10-08_02-17-57:CRCW121010R0FKEAHP
- removed R9: 10 Ohm, CRCW121010R0FKEAHP:RC1210N_VIS-L, symbol 2024-10-08_02-17-57:CRCW121010R0FKEAHP
- removed TP18: Cell 10, TestPoint:TestPoint_Keystone_5010-5014_Multipurpose, symbol Connector:TestPoint
- removed TP19: Cell 9, TestPoint:TestPoint_Keystone_5010-5014_Multipurpose, symbol Connector:TestPoint
- removed TP20: Cell 8, TestPoint:TestPoint_Keystone_5010-5014_Multipurpose, symbol Connector:TestPoint
- removed TP21: Cell 7, symbol Connector:TestPoint
- removed TP22: Cell 6, TestPoint:TestPoint_Keystone_5010-5014_Multipurpose, symbol Connector:TestPoint
- removed TP23: Cell 5, TestPoint:TestPoint_Keystone_5010-5014_Multipurpose, symbol Connector:TestPoint
- removed TP24: Cell 4, TestPoint:TestPoint_Keystone_5010-5014_Multipurpose, symbol Connector:TestPoint
- removed TP25: Cell 3, TestPoint:TestPoint_Keystone_5010-5014_Multipurpose, symbol Connector:TestPoint
- removed TP26: Cell 2, TestPoint:TestPoint_Keystone_5010-5014_Multipurpose, symbol Connector:TestPoint
- removed TP27: Cell 1, TestPoint:TestPoint_Keystone_5010-5014_Multipurpose, symbol Connector:TestPoint
- removed TP28: Cell 0S, TestPoint:TestPoint_Keystone_5010-5014_Multipurpose, symbol Connector:TestPoint
- removed TP29: Cell 14, TestPoint:TestPoint_Keystone_5010-5014_Multipurpose, symbol Connector:TestPoint
- removed TP30: Cell 13, TestPoint:TestPoint_Keystone_5010-5014_Multipurpose, symbol Connector:TestPoint
- removed TP31: Cell 12, TestPoint:TestPoint_Keystone_5010-5014_Multipurpose, symbol Connector:TestPoint
- removed TP32: Cell 11, TestPoint:TestPoint_Keystone_5010-5014_Multipurpose, symbol Connector:TestPoint
- added R10, R4, R5: 7.5 ohm, CRCW12067R50FKEAHP:RES_V1206_VIS-L, symbol 2024-10-28_23-49-19:CRCW12067R50FKEAHP
- added R11, R12, R2, R24, R25, R26, R27, R3, R6, R7, R8, R9: 7.5 Ohm, CRCW12067R50FKEAHP:RES_V1206_VIS-L, symbol 2024-10-28_23-49-19:CRCW12067R50FKEAHP
- added TP18, TP19, TP20, TP21, TP22, TP23, TP24, TP25, TP26, TP27, TP28, TP29, TP30, TP31: 5012, TP5012:TP_5012, symbol 5012:5012
- added TP32: 5011, 5011 (1):TP_5011, symbol 5011:5011
- C10, C11, C12, C13, C14, C15, C16, C17, C18, C19, C20, C21, C22, C23, C24, C25, C26, C27, C28, C29, C30, C31, C32, C33, C35, C36, C37, C38, C9: footprint Capacitor_SMD:C_0201_0603Metric -> GCM188R71C474KA55D:G-188_MUR-L
- C34: footprint Capacitor_SMD:C_0603_1608Metric -> GCM188R71C474KA55D:G-188_MUR-L
- R13, R14, R15, R16, R17, R18, R19, R20, R21, R22, R23, R28, R29, R30, R31: footprint Resistor_SMD:R_0201_0603Metric -> ERA-3AEB101V:RC0603N_PAN-L
Connections:
- net CB0: now also R12.1
- net CB1: now also R11.1
- net CB10: now also R2.1
- net CB11: now also R24.1
- net CB12: now also R25.1
- net CB13: now also R26.1
- net CB14: now also R27.1
- net CB2: now also R10.1
- net CB3: now also R9.1
- net CB4: now also R8.1
- net CB5: now also R7.1
- net CB6: now also R6.1
- net CB7: now also R5.1
- net CB8: now also R4.1
- net CB9: now also R3.1
- net Cell 0: now also R12.2, TP32.TP
- net Cell 1: now also R11.2, TP27.TP
- net Cell 10: now also R2.2, TP18.TP
- net Cell 11: now also R24.2, TP28.TP
- net Cell 12: now also R25.2, TP29.TP
- net Cell 13: now also R26.2, TP30.TP
- net Cell 14S: now also R27.2, TP31.TP
- net Cell 2: now also R10.2, TP26.TP
- net Cell 3: now also R9.2, TP25.TP
- net Cell 4: now also R8.2, TP24.TP
- net Cell 5: now also R7.2, TP23.TP
- net Cell 6: now also R6.2, TP22.TP
- net Cell 7: now also R5.2, TP21.TP
- net Cell 8: now also R4.2, TP20.TP
- net Cell 9: now also R3.2, TP19.TP
