File: DaughterBoard/untitled.kicad_sch (KiCad schematic)
At the start: 75 parts

Commit message: Daughter Update
Connections:
- net GND_AVSS renamed GND

Commit message: 11/9/2024
Changed lines of the file:
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@@
 		)
 	)
-	(global_label "GND_AVSS"
+	(global_label "AVSS"
 		(shape input)
 		(at 210.82 370.84 0)
@@
 		)
 		(property "Intersheetrefs" "${INTERSHEET_REFS}"
-			(at 223.2395 370.84 0)
+			(at 218.4014 370.84 0)
 			(effects
 				(font
@@
 		)
 	)
-	(global_label "GND_AVSS"
+	(global_label "AVSS"
 		(shape input)
 		(at 170.18 386.08 0)
@@
 		)
 		(property "Intersheetrefs" "${INTERSHEET_REFS}"
-			(at 182.5995 386.08 0)
-			(effects
-				(font
+			(at 177.7614 386.08 0)
+			(effects
+				(font

Commit message: DOBO ERC 139 warnings left
Parts:
- TP32: footprint 5011 (1):TP_5011 -> 5011:TP_5011
Changed lines of the file:
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@@
 			)
 		)
-		(property "Footprint" "5011 (1):TP_5011"
+		(property "Footprint" "5011:TP_5011"
 			(at 142.24 349.25 0)
 			(effects

Commit message: Fuse
Parts:
- added F1, F10, F11, F12, F13, F14, F15, F2, F3, F4, F5, F6, F7, F8, F9: 0686F1000-01, 0686F1000-01:FUSC1608X60N, symbol 0686F1000-01:0686F1000-01
- added F16, F17, F18, F19, F20, F21, F22, F23, F24, F25, F26, F27, F28, F29, F30: 0438.250WRA, FUSC1608X61N, symbol 0438_250WRA:0438.250WRA
Connections:
- net Cell 0: now also F16.1; no longer R12.2, R23.2, TP32.TP
- net Cell 1: now also F17.1; no longer R11.2, R22.2, TP27.TP
- net Cell 10: now also F26.1; no longer R13.2, R2.2, TP18.TP
- net Cell 11: now also F27.1; no longer R24.2, R31.2, TP28.TP
- net Cell 12: now also F28.1; no longer R25.2, R30.2, TP29.TP
- net Cell 13: now also F29.1; no longer R26.2, R29.2, TP30.TP
- net Cell 14S: now also F30.1; no longer R27.2, R28.2, TP31.TP
- net Cell 2: now also F18.1; no longer R10.2, R21.2, TP26.TP
- net Cell 3: now also F19.1; no longer R20.2, R9.2, TP25.TP
- net Cell 4: now also F20.1; no longer R19.2, R8.2, TP24.TP
- net Cell 5: now also F21.1; no longer R18.2, R7.2, TP23.TP
- net Cell 6: now also F22.1; no longer R17.2, R6.2, TP22.TP
- net Cell 7: now also F23.1; no longer R16.2, R5.2, TP21.TP
- net Cell 8: now also F24.1; no longer R15.2, R4.2, TP20.TP
- net Cell 9: now also F25.1; no longer R14.2, R3.2, TP19.TP
- new net: F7.2, R17.2, R6.2, TP22.TP
- new net: F13.2, R25.2, R30.2, TP29.TP
- new net: F2.2, R11.2, R22.2, TP27.TP
- new net: F12.1, F27.2
- new net: F12.2, R24.2, R31.2, TP28.TP
- new net: F13.1, F28.2
- new net: F21.2, F6.1
- new net: F6.2, R18.2, R7.2, TP23.TP
- new net: F4.2, R20.2, R9.2, TP25.TP
- new net: F14.2, R26.2, R29.2, TP30.TP
- new net: F10.1, F25.2
- new net: F10.2, R14.2, R3.2, TP19.TP
- new net: F18.2, F3.1
- new net: F3.2, R10.2, R21.2, TP26.TP
- new net: F1.1, F16.2
- new net: F11.2, R13.2, R2.2, TP18.TP
- new net: F14.1, F29.2
- new net: F17.2, F2.1
- new net: F22.2, F7.1
- new net: F5.2, R19.2, R8.2, TP24.TP
- new net: F23.2, F8.1
- new net: F11.1, F26.2
- new net: F9.2, R15.2, R4.2, TP20.TP
- new net: F20.2, F5.1
- new net: F15.1, F30.2
- new net: F15.2, R27.2, R28.2, TP31.TP
- new net: F1.2, R12.2, R23.2, TP32.TP
- new net: F19.2, F4.1
- new net: F8.2, R16.2, R5.2, TP21.TP
- new net: F24.2, F9.1
Other:
- moved on the sheet: C31, C32, C33, C34, C35, C36, C37, C38, R24, R25, R26, R27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

Commit message: Starting Routing
Connections:
- net CB1: now also R11.2; no longer R11.1
- net CB10: now also R2.2; no longer R2.1
- net CB11: now also R24.2; no longer R24.1
- net CB12: now also R25.2; no longer R25.1
- net CB13: now also R26.2; no longer R26.1
- net CB14: now also R27.2; no longer R27.1
- net CB2: now also R10.2; no longer R10.1
- net CB3: now also R9.2; no longer R9.1
- net CB4: now also R8.2; no longer R8.1
- net CB5: now also R7.2; no longer R7.1
- net CB6: now also R6.2; no longer R6.1
- net CB7: now also R5.2; no longer R5.1
- net CB8: now also R4.2; no longer R4.1
- net CB9: now also R3.2; no longer R3.1
- net VC14: now also R28.2; no longer R28.1
- net at F7.2, R17.2, TP22.TP: now also R6.1; no longer R6.2
- net at F13.2, R30.2, TP29.TP: now also R25.1; no longer R25.2
- net at F2.2, R22.2, TP27.TP: now also R11.1; no longer R11.2
- net at F12.2, R31.2, TP28.TP: now also R24.1; no longer R24.2
- net at F6.2, R18.2, TP23.TP: now also R7.1; no longer R7.2
- net at F4.2, R20.2, TP25.TP: now also R9.1; no longer R9.2
- net at F14.2, R29.2, TP30.TP: now also R26.1; no longer R26.2
- net at F10.2, R14.2, TP19.TP: now also R3.1; no longer R3.2
- net at F3.2, R21.2, TP26.TP: now also R10.1; no longer R10.2
- net at F11.2, R13.2, TP18.TP: now also R2.1; no longer R2.2
- net at F5.2, R19.2, TP24.TP: now also R8.1; no longer R8.2
- net at F9.2, R15.2, TP20.TP: now also R4.1; no longer R4.2
- net at F15.2, TP31.TP: now also R27.1, R28.1; no longer R27.2, R28.2
- net at F8.2, R16.2, TP21.TP: now also R5.1; no longer R5.2
Other:
- moved on the sheet: R10, R11, R12, R2, R24, R25, R26, R27, R28, R3, R4, R5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

Commit message: C:/Program Files/Git/
Parts:
- F1, F10, F11, F12, F13, F14, F15, F2, F3, F4, F5, F6, F7, F8, F9: Manufacturer Part Number (none) -> FUSC1608X60N
- F16, F17, F18, F19, F20, F21, F22, F23, F24, F25, F26, F27, F28, F29, F30: Manufacturer Part Number (none) -> FUSC1608X61N
- R10, R11, R12, R2, R24, R25, R26, R27, R3, R4, R5, R6, R7, R8, R9: Manufacturer Part Number (none) -> CRCW12067R50FKEAHP
- TP18, TP19, TP20, TP21, TP22, TP23, TP24, TP25, TP26, TP27, TP28, TP29, TP30, TP31: Manufacturer Part Number (none) -> 5012
- TP32: Manufacturer Part Number (none) -> 5011
