File: DaughterBoard/untitled.kicad_sch (KiCad schematic)
At the start: 105 parts

Commit message: Layout continued. Fixed Footprint and most 3d model
Parts:
- TP32: footprint 5011:TP_5011 -> 5011 (1):TP_5011
Connections:
- net VC0: now also R23.2; no longer R23.1
- net at F1.2, R12.2, TP32.TP: now also R23.1; no longer R23.2
Other:
- moved on the sheet: R23
Changed lines of the file:
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@@
 	)
 	(junction
-		(at 200.66 354.33)
-		(diameter 0)
-		(color 0 0 0 0)
-	)
-	(junction
 		(at 421.64 182.88)
 		(diameter 0)
@@
 	)
 	(junction
-		(at 163.83 241.3)
+		(at 176.53 354.33)
 		(diameter 0)
 		(color 0 0 0 0)
 	)
 	(junction
-		(at 401.32 182.88)
+		(at 163.83 241.3)
 		(diameter 0)
 		(color 0 0 0 0)
 	)
 	(junction
-		(at 176.53 354.33)
+		(at 401.32 182.88)
 		(diameter 0)
 		(color 0 0 0 0)
@@
 	)
 	(junction
+		(at 167.64 354.33)
+		(diameter 0)
+		(color 0 0 0 0)
+	)
+	(junction
 		(at 163.83 170.18)
 		(diameter 0)
@@
 	)
 	(junction
+		(at 200.66 354.33)
+		(diameter 0)
+		(color 0 0 0 0)
+	)
+	(junction
 		(at 401.32 238.76)
 		(diameter 0)
@@
 	(wire
 		(pts
-			(xy 142.24 354.33) (xy 176.53 354.33)
+			(xy 142.24 354.33) (xy 167.64 354.33)
 		)
 		(stroke
@@
 	(wire
 		(pts
+			(xy 167.64 353.06) (xy 167.64 354.33)
+		)
+		(stroke
+			(width 0)
+			(type default)
+		)
+	)
+	(wire
+		(pts
 			(xy 421.64 209.55) (xy 415.29 209.55)
 		)
@@
 	(wire
 		(pts
-			(xy 450.85 210.82) (xy 458.47 210.82)
+			(xy 167.64 354.33) (xy 176.53 354.33)
 		)
 		(stroke
@@
 	(wire
 		(pts
-			(xy 193.04 354.33) (xy 200.66 354.33)
+			(xy 450.85 210.82) (xy 458.47 210.82)
 		)
 		(stroke
@@
 	(wire
 		(pts
-			(xy 176.53 354.33) (xy 180.34 354.33)
-		)
-		(stroke
-			(width 0)
-			(type default)
-		)
-	)
-	(wire
-		(pts
 			(xy 143.51 129.54) (xy 163.83 129.54)
 		)
@@
 	(wire
 		(pts
+			(xy 176.53 354.33) (xy 180.34 354.33)
+		)
+		(stroke
+			(width 0)
+			(type default)
+		)
+	)
+	(wire
+		(pts
 			(xy 130.81 129.54) (xy 143.51 129.54)
 		)
@@
 	(wire
 		(pts
+			(xy 193.04 354.33) (xy 200.66 354.33)
+		)
+		(stroke
+			(width 0)
+			(type default)
+		)
+	)
+	(wire
+		(pts
 			(xy 163.83 101.6) (xy 163.83 109.22)
 		)
@@
 			)
 		)
-		(property "Footprint" "5011:TP_5011"
+		(property "Footprint" "5011 (1):TP_5011"
 			(at 142.24 342.9 0)
 			(effects
@@
 		(lib_name "ERA-3AEB101V_11")
 		(lib_id "2024-10-08_02-28-54:ERA-3AEB101V")
-		(at 180.34 354.33 0)
+		(at 193.04 354.33 180)
 		(unit 1)
 		(exclude_from_sim no)
@@
 		)
 		(property "Footprint" "ERA-3AEB101V:RC0603N_PAN-L"
-			(at 180.848 360.68 0)
+			(at 192.532 347.98 0)
 			(effects
 				(font
@@
 		)
 		(property "Datasheet" ""
-			(at 179.832 357.378 0)
+			(at 193.548 351.282 0)
 			(effects
 				(font
@@
 		)
 		(property "Description" ""
-			(at 180.34 354.33 0)
+			(at 193.04 354.33 0)
 			(effects
 				(font
@@
 		)
 		(property "Manufacturer Part Number" "ERA-3AEB101V"
-			(at 180.086 362.966 0)
+			(at 193.294 345.694 0)
 			(effects
 				(font

Commit message: tracing left
Parts:
- F16, F17, F18, F19, F20, F21, F22, F23, F24, F25, F26, F27, F28, F29, F30: footprint FUSC1608X61N -> 0438.250WRA:FUSC1608X61N
- R10, R4, R5: value 7.5 ohm -> 7.5
- R11, R12, R2, R24, R25, R26, R27, R3, R6, R7, R8, R9: value 7.5 Ohm -> 7.5
- R13, R14, R15, R16, R17, R18, R19, R20, R21, R22, R23, R28, R29, R30, R31: value 100 Ohm -> 100
- TP18, TP19, TP20, TP21, TP22, TP23, TP24, TP25, TP26, TP27, TP28, TP29, TP30, TP31: footprint TP5012:TP_5012 -> 5012:TP_5012

Commit message: Routing Update 3
Parts:
- R10, R11, R12, R2, R24, R25, R26, R27, R3, R4, R5, R6, R7, R8, R9: value 7.5 -> 7.5
- R13, R14, R15, R16, R17, R18, R19, R20, R21, R22, R23, R28, R29, R30, R31: value 100 -> 100
Connections:
- net GND renamed GND_AVSS
Changed lines of the file:
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@@
 			)
 		)
-		(property "Value" "100 "
+		(property "Value" "100"
 			(at 186.69 181.61 0)
 			(effects
@@
 			)
 		)
-		(property "Value" "100 "
+		(property "Value" "100"
 			(at 444.5 234.95 0)
 			(effects
@@
 			)
 		)
-		(property "Value" "7.5 "
+		(property "Value" "7.5"
 			(at 170.18 328.93 0)
 			(effects
@@
 			)
 		)
-		(property "Value" "7.5 "
+		(property "Value" "7.5"
 			(at 170.18 273.05 0)
 			(effects
@@
 			)
 		)
-		(property "Value" "7.5 "
+		(property "Value" "7.5"
 			(at 427.99 214.63 0)
 			(effects
@@
 			)
 		)
-		(property "Value" "100 "
+		(property "Value" "100"
 			(at 186.69 321.31 0)
 			(effects
@@
 			)
 		)
-		(property "Value" "7.5 "
+		(property "Value" "7.5"
 			(at 170.18 300.99 0)
 			(effects
@@
 			)
 		)
-		(property "Value" "7.5 "
+		(property "Value" "7.5"
 			(at 170.18 77.47 0)
 			(effects
@@
 			)
 		)
-		(property "Value" "7.5 "
+		(property "Value" "7.5"
 			(at 170.18 190.5 0)
 			(effects
@@
 			)
 		)
-		(property "Value" "100 "
+		(property "Value" "100"
 			(at 444.5 262.89 0)
 			(effects
@@
 		(on_board yes)
 		(dnp no)
-		(fields_autoplaced yes)
 		(property "Reference" "#PWR07"
 			(at 204.47 378.46 0)
@@
 			)
 		)
-		(property "Value" "GND"
-			(at 204.47 377.19 0)
+		(property "Value" "GND_AVSS"
+			(at 199.644 379.222 0)
 			(effects
 				(font
 					(size 1.27 1.27)
 				)
+				(justify left)
 			)
 		)
@@
 			)
 		)
-		(property "Value" "100 "
+		(property "Value" "100"
 			(at 186.69 69.85 0)
 			(effects
@@
 			)
 		)
-		(property "Value" "7.5 "
+		(property "Value" "7.5"
 			(at 430.53 273.05 0)
 			(effects
@@
 			)
 		)
-		(property "Value" "7.5 "
+		(property "Value" "7.5"
 			(at 170.18 245.11 0)
 			(effects
@@
 			)
 		)
-		(property "Value" "7.5 "
+		(property "Value" "7.5"
 			(at 170.18 133.35 0)
 			(effects
@@
 			)
 		)
-		(property "Value" "7.5 "
+		(property "Value" "7.5"
 			(at 170.18 218.44 0)
 			(effects
@@
 			)
 		)
-		(property "Value" "100 "
+		(property "Value" "100"
 			(at 186.69 265.43 0)
 			(effects
@@
 			)
 		)
-		(property "Value" "100 "
+		(property "Value" "100"
 			(at 186.69 97.79 0)
 			(effects
@@
 			)
 		)
-		(property "Value" "7.5 "
+		(property "Value" "7.5"
 			(at 430.53 243.84 0)
 			(effects
@@
 			)
 		)
-		(property "Value" "7.5 "
+		(property "Value" "7.5"
 			(at 170.18 363.22 0)
 			(effects
@@
 			)
 		)
-		(property "Value" "100 "
+		(property "Value" "100"
 			(at 186.69 293.37 0)
 			(effects
@@
 			)
 		)
-		(property "Value" "100 "
+		(property "Value" "100"
 			(at 186.69 153.67 0)
 			(effects
@@
 			)
 		)
-		(property "Value" "7.5 "
+		(property "Value" "7.5"
 			(at 427.99 187.96 0)
 			(effects
@@
 			)
 		)
-		(property "Value" "7.5 "
+		(property "Value" "7.5"
 			(at 170.18 161.29 0)
 			(effects
@@
 			)
 		)
-		(property "Value" "100 "
+		(property "Value" "100"
 			(at 186.69 237.49 0)
 			(effects
@@
 		(on_board yes)
 		(dnp no)
-		(fields_autoplaced yes)
 		(property "Reference" "#PWR06"
 			(at 163.83 393.7 0)
@@
 			)
 		)
-		(property "Value" "GND"
-			(at 163.83 392.43 0)
+		(property "Value" "GND_AVSS"
+			(at 158.75 392.684 0)
 			(effects
 				(font
 					(size 1.27 1.27)
 				)
+				(justify left)
 			)
 		)
@@
 			)
 		)
-		(property "Value" "100 "
+		(property "Value" "100"
 			(at 444.5 207.01 0)
 			(effects
@@
 			)
 		)
-		(property "Value" "100 "
+		(property "Value" "100"
 			(at 444.5 179.07 0)
 			(effects
@@
 			)
 		)
-		(property "Value" "7.5 "
+		(property "Value" "7.5"
 			(at 170.18 105.41 0)
 			(effects
@@
 			)
 		)
-		(property "Value" "100 "
+		(property "Value" "100"
 			(at 186.69 350.52 0)
 			(effects
@@
 			)
 		)
-		(property "Value" "100 "
+		(property "Value" "100"
 			(at 186.69 125.73 0)
 			(effects
@@
 			)
 		)
-		(property "Value" "100 "
+		(property "Value" "100"
 			(at 186.69 209.55 0)
 			(effects

Commit message: Updates
Connections:
- net GND_AVSS renamed GND
Changed lines of the file:
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@@
 	(symbol
 		(lib_id "power:GND")
-		(at 204.47 372.11 0)
+		(at 163.83 387.35 0)
 		(unit 1)
 		(exclude_from_sim no)
@@
 		(on_board yes)
 		(dnp no)
-		(property "Reference" "#PWR07"
-			(at 204.47 378.46 0)
+		(fields_autoplaced yes)
+		(property "Reference" "#PWR02"
+			(at 163.83 393.7 0)
 			(effects
 				(font
@@
 			)
 		)
-		(property "Value" "GND_AVSS"
-			(at 199.644 379.222 0)
+		(property "Value" "GND"
+			(at 163.83 392.43 0)
 			(effects
 				(font
 					(size 1.27 1.27)
 				)
-				(justify left)
 			)
 		)
 		(property "Footprint" ""
-			(at 204.47 372.11 0)
+			(at 163.83 387.35 0)
 			(effects
 				(font
@@
 		)
 		(property "Datasheet" ""
-			(at 204.47 372.11 0)
+			(at 163.83 387.35 0)
 			(effects
 				(font
@@
 		)
 		(property "Description" "Power symbol creates a global label with name \"GND\" , ground"
-			(at 204.47 372.11 0)
+			(at 163.83 387.35 0)
 			(effects
 				(font
@@
 			(project "Project63_BMS_DaughterBoard"
 				(path "/325b096d-8e4c-4cdc-b4c5-634ea5e73c60/2fc75a92-430f-42ad-9ad5-d910a7d34c12"
-					(reference "#PWR07")
+					(reference "#PWR02")
 					(unit 1)
 				)
@@
 	)
 	(symbol
+		(lib_id "power:GND")
+		(at 204.47 372.11 0)
+		(unit 1)
+		(exclude_from_sim no)
+		(in_bom yes)
+		(on_board yes)
+		(dnp no)
+		(fields_autoplaced yes)
+		(property "Reference" "#PWR03"
+			(at 204.47 378.46 0)
+			(effects
+				(font
+					(size 1.27 1.27)
+				)
+				(hide yes)
+			)
+		)
+		(property "Value" "GND"
+			(at 204.47 377.19 0)
+			(effects
+				(font
+					(size 1.27 1.27)
+				)
+			)
+		)
+		(property "Footprint" ""
+			(at 204.47 372.11 0)
+			(effects
+				(font
+					(size 1.27 1.27)
+				)
+				(hide yes)
+			)
+		)
+		(property "Datasheet" ""
+			(at 204.47 372.11 0)
+			(effects
+				(font
+					(size 1.27 1.27)
+				)
+				(hide yes)
+			)
+		)
+		(property "Description" "Power symbol creates a global label with name \"GND\" , ground"
+			(at 204.47 372.11 0)
+			(effects
+				(font
+					(size 1.27 1.27)
+				)
+				(hide yes)
+			)
+		)
+		(pin "1"
+		)
+		(instances
+			(project "Project63_BMS_DaughterBoard"
+				(path "/325b096d-8e4c-4cdc-b4c5-634ea5e73c60/2fc75a92-430f-42ad-9ad5-d910a7d34c12"
+					(reference "#PWR03")
+					(unit 1)
+				)
+			)
+		)
+	)
+	(symbol
 		(lib_name "CRCW12067R50FKEAHP_3")
 		(lib_id "2024-10-28_23-49-19:CRCW12067R50FKEAHP")
@@
 					(unit 1)
 				)
-			)
-		)
-	)
-	(symbol
-		(lib_id "power:GND")
-		(at 163.83 387.35 0)
-		(unit 1)
-		(exclude_from_sim no)
-		(in_bom yes)
-		(on_board yes)
-		(dnp no)
-		(property "Reference" "#PWR06"
-			(at 163.83 393.7 0)
-			(effects
-				(font
-					(size 1.27 1.27)
-				)
-				(hide yes)
-			)
-		)
-		(property "Value" "GND_AVSS"
-			(at 158.75 392.684 0)
-			(effects
-				(font
-					(size 1.27 1.27)
-				)
-				(justify left)
-			)
-		)
-		(property "Footprint" ""
-			(at 163.83 387.35 0)
-			(effects
-				(font
-					(size 1.27 1.27)
-				)
-				(hide yes)
-			)
-		)
-		(property "Datasheet" ""
-			(at 163.83 387.35 0)
-			(effects
-				(font
-					(size 1.27 1.27)
-				)
-				(hide yes)
-			)
-		)
-		(property "Description" "Power symbol creates a global label with name \"GND\" , ground"
-			(at 163.83 387.35 0)
-			(effects
-				(font
-					(size 1.27 1.27)
-				)
-				(hide yes)
-			)
-		)
-		(pin "1"
-		)
-		(instances
-			(project "Project63_BMS_DaughterBoard"
-				(path "/325b096d-8e4c-4cdc-b4c5-634ea5e73c60/2fc75a92-430f-42ad-9ad5-d910a7d34c12"
-					(reference "#PWR06")
-					(unit 1)
-				)

Commit message: Finished board
Parts:
- renumbered C9 to C301, C10 to C302, C11 to C303, C12 to C304, C13 to C305, C14 to C306, C15 to C307, C16 to C308, C17 to C309, C18 to C310, C19 to C311, C20 to C312, C21 to C313, C22 to C314, C23 to C315, C24 to C316, C25 to C317, C26 to C318, C27 to C319, C28 to C320, C29 to C321, C30 to C322, C31 to C323, C32 to C324, C33 to C325, C34 to C326, C35 to C327, C36 to C328, C37 to C329, C38 to C330, F26 to F301, F25 to F302, F24 to F303, F23 to F304, F22 to F305, F21 to F306, F20 to F307, F19 to F308, F18 to F309, F17 to F310, F16 to F311, F11 to F312, F10 to F313, F9 to F314, F8 to F315, F7 to F316, F2 to F317, F6 to F318, F5 to F319, F4 to F320, F3 to F321, F1 to F322, F30 to F323, F29 to F324, F28 to F325, F27 to F326, F15 to F327, F14 to F328, F13 to F329, F12 to F330, R2 to R301, R3 to R302, R4 to R303, R5 to R304, R6 to R305, R7 to R306, R8 to R307, R9 to R308, R10 to R309, R11 to R310, R12 to R311, R13 to R312, R14 to R313, R15 to R314, R16 to R315, R17 to R316, R18 to R317, R19 to R318, R20 to R319, R21 to R320, R22 to R321, R23 to R322, R27 to R323, R26 to R324, R25 to R325, R24 to R326, R29 to R327, R30 to R328, R31 to R329, R28 to R330, TP32 to TP301, TP18 to TP302, TP19 to TP303, TP20 to TP304, TP21 to TP305, TP22 to TP306, TP23 to TP307, TP24 to TP308, TP25 to TP309, TP26 to TP310, TP27 to TP311, TP31 to TP312, TP30 to TP313, TP29 to TP314, TP28 to TP315

Commit message: Daughterboard 100% Complete + Edited Motherboard BOM
Parts:
- F301, F302, F303, F304, F305, F306, F307, F308, F309, F310, F311, F323, F324, F325, F326: footprint 0438.250WRA:FUSC1608X61N -> Fuse:Fuse_0603_1608Metric
- renumbered TP312 to BAT_POSITIVE301, TP313 to TP312, TP314 to TP313, TP315 to TP314
Connections:
- net Cell 0 renamed Cell 0S

Commit message: Both boards complete
Parts:
- BAT_POSITIVE301, TP301, TP302, TP303, TP304, TP305, TP306, TP307, TP308, TP309, TP310, TP311, TP312, TP313, TP314: now not fitted
- C301, C302, C303, C304, C305, C306, C307, C308, C309, C310, C311, C312, C313, C314, C315, C316, C317, C318, C319, C320, C321, C322, C323, C324, C325, C326, C327, C328, C329, C330: JLC PCB Part # (none) -> C161214
- F301, F302, F303, F304, F305, F306, F307, F308, F309, F310, F311, F323, F324, F325, F326: JLC PCB Part # (none) -> C151137; Manufacturer Part Number FUSC1608X61N -> 0467.250NRHF
- F312, F313, F314, F315, F316, F317, F318, F319, F320, F321, F322, F327, F328, F329, F330: JLC PCB Part # (none) -> C136329; Manufacturer Part Number FUSC1608X60N -> JFC0603-1100FS
- R301, R302, R303, R304, R305, R306, R307, R308, R309, R310, R311, R323, R324, R325, R326: footprint CRCW12067R50FKEAHP:RES_V1206_VIS-L -> Resistor_SMD:R_1812_4532Metric; JLC PCB Part # (none) -> C5204035; Manufacturer Part Number CRCW12067R50FKEAHP -> FRC1812J7R5 TS
- R312, R313, R314, R315, R316, R317, R318, R319, R320, R321, R322, R327, R328, R329, R330: footprint ERA-3AEB101V:RC0603N_PAN-L -> Resistor_SMD:R_0603_1608Metric; JLC PCB Part # (none) -> C5123580; Manufacturer Part Number ERA-3AEB101V -> HoAR0603-1/10W-100R-0.1%-TCR25
