File: DaughterBoard/NPN Power Supply.kicad_sch (KiCad schematic)
At the start: 4 parts, among them Q1 2n2222

Commit message: 90% DOBO is done
Parts:
- removed C40: 0.22, Capacitor_SMD:C_1206_3216Metric, symbol Device:C
- removed Q1: 2n2222, OptoDevice:Osram_SFH3710, symbol Transistor_BJT:FFB2222A
- removed R40: 100, Resistor_SMD:R_2010_5025Metric, symbol Device:R_US
- removed R41: 200, Resistor_SMD:R_2010_5025Metric, symbol Device:R_US

Commit message: NPN is done
Parts:
- added C39: 0.22µF, GCM31MR72A224KA3L:G-31_MUR-L, symbol GCM31MR72A224KA37L:GCM31MR72A224KA37L
- added Q1: ZXTN4004KTC, ZXTN4004KTC:ZXTN4004KTC, symbol ZXTN4004KTC:ZXTN4004KTC
- added R32: 100, CRCW2010100RFKEF:RES_CRCW_2010-L, symbol CRCW2010100RFKEF:CRCW2010100RFKEF
- added R33: 200, CRCW2010200RFKEF:RC2010N_VIS-L, symbol CRCW2010200RFKEF:CRCW2010200RFKEF
Connections:
- net GND: now also C39.2
- net LDOIN: now also Q1.3 (E)
- net NPNB: now also Q1.1 (B)
- net PWR: now also R33.2
- new net: C39.1, Q1.2 (C), R32.2
- new net: R32.1, R33.1
