File: DaughterBoard/NPN Power Supply.kicad_sch (KiCad schematic)
At the start: 4 parts, among them Q1 ZXTN4004KTC

Commit message: 11/9/2024
Connections:
- net PWR renamed Cell 14S
Changed lines of the file:
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@@
 	(wire
 		(pts
-			(xy 196.85 106.68) (xy 213.36 106.68)
+			(xy 196.85 106.68) (xy 222.25 106.68)
 		)
 		(stroke
@@
 		)
 	)
-	(global_label "PWR"
+	(global_label "Cell 14S"
 		(shape input)
-		(at 213.36 106.68 0)
+		(at 222.25 106.68 0)
 		(fields_autoplaced yes)
 		(effects
@@
 		)
 		(property "Intersheetrefs" "${INTERSHEET_REFS}"
-			(at 220.3366 106.68 0)
+			(at 233.5203 106.68 0)
 			(effects
 				(font

Commit message: DOBO ERC 139 warnings left
Parts:
- C39: footprint GCM31MR72A224KA3L:G-31_MUR-L -> G-31_MUR
- Q1: footprint ZXTN4004KTC:ZXTN4004KTC -> ZXTN4004KTC
- R32: footprint CRCW2010100RFKEF:RES_CRCW_2010-L -> RES_CRCW_2010
- R33: footprint CRCW2010200RFKEF:RC2010N_VIS-L -> RC2010N_VIS
Changed lines of the file:
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@@
 			)
 		)
-		(property "Footprint" "GCM31MR72A224KA3L:G-31_MUR-L"
+		(property "Footprint" "G-31_MUR"
 			(at 137.414 106.934 0)
 			(effects
@@
 			)
 		)
-		(property "Footprint" "CRCW2010200RFKEF:RC2010N_VIS-L"
+		(property "Footprint" "RC2010N_VIS"
 			(at 184.15 100.33 0)
 			(effects
@@
 			)
 		)
-		(property "Footprint" "ZXTN4004KTC:ZXTN4004KTC"
+		(property "Footprint" "ZXTN4004KTC"
 			(at 90.17 -11.1 0)
 			(effects
@@
 			)
 		)
-		(property "Footprint" "CRCW2010100RFKEF:RES_CRCW_2010-L"
+		(property "Footprint" "RES_CRCW_2010"
 			(at 150.622 100.584 0)
 			(effects

Commit message: C:/Program Files/Git/
Parts:
- C39: Manufacturer Part Number (none) -> GCM31MR72A224KA37L
- Q1: Manufacturer Part Number (none) -> ZXTN4004KTC
- R32: Manufacturer Part Number (none) -> CRCW2010100RFKEF
- R33: Manufacturer Part Number (none) -> CRCW2010200RFKEF
Changed lines of the file:
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@@
+			)
+		)
+		(property "Manufacturer Part Number" "GCM31MR72A224KA37L"
+			(at 133.35 106.68 0)
+			(effects
+				(font
+					(size 1.27 1.27)
+				)
+				(hide yes)
 			)
 		)
@@
 			)
 		)
+		(property "Manufacturer Part Number" "CRCW2010200RFKEF"
+			(at 184.15 106.68 0)
+			(effects
+				(font
+					(size 1.27 1.27)
+				)
+				(hide yes)
+			)
+		)
 		(pin "2"
 		)
@@
 			)
 		)
+		(property "Manufacturer Part Number" "ZXTN4004KTC"
+			(at 104.14 90.17 0)
+			(effects
+				(font
+					(size 1.27 1.27)
+				)
+				(hide yes)
+			)
+		)
 		(pin "3"
 		)
@@
 			(at 149.86 106.68 0)
 			(effects
+				(font
+					(size 1.27 1.27)
+				)
+				(hide yes)
+			)
+		)
+		(property "Manufacturer Part Number" "CRCW2010100RFKEF"
+			(at 149.86 106.68 0)
+			(effects
