File: DaughterBoard/NPN Power Supply.kicad_sch (KiCad schematic)
At the start: 4 parts, among them Q1 ZXTN4004KTC

Commit message: Layout continued. Fixed Footprint and most 3d model
Parts:
- C39: footprint G-31_MUR -> GCM31MR72A224KA37L:G-31_MUR-L
- R32: footprint RES_CRCW_2010 -> CRCW2010100RFKEF:RES_CRCW_2010-L
Changed lines of the file:
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@@
 			)
 		)
-		(property "Footprint" "G-31_MUR"
+		(property "Footprint" "GCM31MR72A224KA37L:G-31_MUR-L"
 			(at 137.414 106.934 0)
 			(effects
@@
 			)
 		)
-		(property "Footprint" "RES_CRCW_2010"
+		(property "Footprint" "CRCW2010100RFKEF:RES_CRCW_2010-L"
 			(at 150.622 100.584 0)
 			(effects

Commit message: tracing left
Parts:
- Q1: footprint ZXTN4004KTC -> ZXTN4004KTC:ZXTN4004KTC
- R32: value 100 -> 100
- R33: value 200 -> 200; footprint RC2010N_VIS -> CRCW2010200RFKEF:RC2010N_VIS-L
Changed lines of the file:
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@@
 			)
 		)
-		(property "Datasheet" ""
+		(property "Datasheet" "https://search.murata.co.jp/Ceramy/image/img/A01X/G101/ENG/GCM033R71A103KA03-01A.pdf"
 			(at 137.414 106.934 0)
 			(effects
@@
 			)
 		)
-		(property "Value" "200"
+		(property "Value" "200 "
 			(at 190.5 110.49 0)
 			(effects
@@
 			)
 		)
-		(property "Footprint" "RC2010N_VIS"
+		(property "Footprint" "CRCW2010200RFKEF:RC2010N_VIS-L"
 			(at 184.15 100.33 0)
 			(effects
@@
 			)
 		)
-		(property "Datasheet" ""
+		(property "Datasheet" "https://www.vishay.com/docs/20035/dcrcwe3.pdf"
 			(at 184.15 100.33 0)
 			(effects
@@
 			)
 		)
-		(property "Footprint" "ZXTN4004KTC"
+		(property "Footprint" "ZXTN4004KTC:ZXTN4004KTC"
 			(at 90.17 -11.1 0)
 			(effects
@@
 			)
 		)
-		(property "Value" "100"
+		(property "Value" "100 "
 			(at 156.21 110.49 0)
 			(effects
@@
 			)
 		)
-		(property "Datasheet" ""
+		(property "Datasheet" "https://www.vishay.com/docs/20035/dcrcwe3.pdf"
 			(at 150.622 100.584 0)
 			(effects

Commit message: Routing Update 3
Parts:
- R32: value 100 -> 100
- R33: value 200 -> 200
Changed lines of the file:
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@@
 			)
 		)
-		(property "Value" "200 "
+		(property "Value" "200"
 			(at 190.5 110.49 0)
 			(effects
@@
 			)
 		)
-		(property "Value" "100 "
+		(property "Value" "100"
 			(at 156.21 110.49 0)
 			(effects

Commit message: Silkscreen edits
Parts:
- C39: value 0.22µF -> 0.22uF
Changed lines of the file:
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@@
 			)
 		)
-		(property "Value" "0.22µF"
+		(property "Value" "0.22uF"
 			(at 129.54 111.7599 90)
 			(effects

Commit message: Finished board
Parts:
- renumbered C39 to C601, Q1 to Q601, R32 to R601, R33 to R602
Changed lines of the file:
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@@
 		(on_board yes)
 		(dnp no)
-		(property "Reference" "C39"
+		(property "Reference" "C601"
 			(at 129.54 109.2199 90)
 			(effects
@@
 			(project "Project63_BMS_DaughterBoard"
 				(path "/325b096d-8e4c-4cdc-b4c5-634ea5e73c60/50508abc-94ca-4760-9b7e-3243f83fc341"
-					(reference "C39")
+					(reference "C601")
 					(unit 1)
 				)
@@
 		(dnp no)
 		(fields_autoplaced yes)
-		(property "Reference" "#PWR01"
+		(property "Reference" "#PWR0601"
 			(at 133.35 120.65 0)
 			(effects
@@
 			(project "Project63_BMS_DaughterBoard"
 				(path "/325b096d-8e4c-4cdc-b4c5-634ea5e73c60/50508abc-94ca-4760-9b7e-3243f83fc341"
-					(reference "#PWR01")
+					(reference "#PWR0601")
 					(unit 1)
 				)
@@
 		(on_board yes)
 		(dnp no)
-		(property "Reference" "R33"
+		(property "Reference" "R602"
 			(at 190.5 113.03 0)
 			(effects
@@
 			(project "Project63_BMS_DaughterBoard"
 				(path "/325b096d-8e4c-4cdc-b4c5-634ea5e73c60/50508abc-94ca-4760-9b7e-3243f83fc341"
-					(reference "R33")
+					(reference "R602")
 					(unit 1)
 				)
@@
 		(dnp no)
 		(fields_autoplaced yes)
-		(property "Reference" "Q1"
+		(property "Reference" "Q601"
 			(at 90.17 88.8999 0)
 			(effects
@@
 			(project "Project63_BMS_DaughterBoard"
 				(path "/325b096d-8e4c-4cdc-b4c5-634ea5e73c60/50508abc-94ca-4760-9b7e-3243f83fc341"
-					(reference "Q1")
+					(reference "Q601")
 					(unit 1)
 				)
@@
 		(on_board yes)
 		(dnp no)
-		(property "Reference" "R32"
+		(property "Reference" "R601"
 			(at 156.21 113.03 0)
 			(effects
@@
 			(project "Project63_BMS_DaughterBoard"
 				(path "/325b096d-8e4c-4cdc-b4c5-634ea5e73c60/50508abc-94ca-4760-9b7e-3243f83fc341"
-					(reference "R32")
+					(reference "R601")
 					(unit 1)
 				)

Commit message: Daughterboard 100% Complete + Edited Motherboard BOM
Connections:
- net Cell 14S renamed Cell 14
Changed lines of the file:
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@@
 		)
 	)
-	(global_label "Cell 14S"
+	(global_label "Cell 14"
 		(shape input)
 		(at 222.25 106.68 0)
@@
 		)
 		(property "Intersheetrefs" "${INTERSHEET_REFS}"
-			(at 233.5203 106.68 0)
+			(at 232.3108 106.68 0)
 			(effects
 				(font

Commit message: Both boards complete
Parts:
- C601: JLC PCB Part # (none) -> C161277
- Q601: JLC PCB Part # (none) -> C157603
- R601: JLC PCB Part # (none) -> C305269; Manufacturer Part Number CRCW2010100RFKEF -> WF20P1000FTL
- R602: footprint CRCW2010200RFKEF:RC2010N_VIS-L -> Resistor_SMD:R_2512_6332Metric; JLC PCB Part # (none) -> C2935248; Manufacturer Part Number CRCW2010200RFKEF -> RC2512JK-07200RL
Changed lines of the file:
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@@
+			)
+		)
+		(property "JLC PCB Part #" "C161277"
+			(at 133.35 106.68 0)
+			(effects
+				(font
+					(size 1.27 1.27)
+				)
+				(hide yes)
 			)
 		)
@@
 			)
 		)
-		(property "Footprint" "CRCW2010200RFKEF:RC2010N_VIS-L"
+		(property "Footprint" "Resistor_SMD:R_2512_6332Metric"
 			(at 184.15 100.33 0)
 			(effects
@@
 			)
 		)
-		(property "Manufacturer Part Number" "CRCW2010200RFKEF"
+		(property "Manufacturer Part Number" "RC2512JK-07200RL"
+			(at 184.15 106.68 0)
+			(effects
+				(font
+					(size 1.27 1.27)
+				)
+				(hide yes)
+			)
+		)
+		(property "JLC PCB Part #" "C2935248"
 			(at 184.15 106.68 0)
 			(effects
@@
 			)
 		)
+		(property "JLC PCB Part #" "C157603"
+			(at 104.14 90.17 0)
+			(effects
+				(font
+					(size 1.27 1.27)
+				)
+				(hide yes)
+			)
+		)
 		(pin "3"
 		)
@@
 			)
 		)
-		(property "Manufacturer Part Number" "CRCW2010100RFKEF"
+		(property "Manufacturer Part Number" "WF20P1000FTL"
 			(at 149.86 106.68 0)
 			(effects
+				(font
+					(size 1.27 1.27)
+				)
+				(hide yes)
+			)
+		)
+		(property "JLC PCB Part #" "C305269"
+			(at 149.86 106.68 0)
+			(effects
