File: DaughterBoard/Project63_BMS_DaughterBoard.kicad_pcb (KiCad board)
At the start: 2 copper layers, 163 parts, among them J1 705550019, J2 705510038, J2 PEC03SAAN, J3 705510038, J3 PEC02SAAN, J4 PEC02SAAN, Q1 ZXTN4004KTC, U1 BQ79614PAPRQ1

Commit message: Fuse
Parts:
- added F1: 0686F1000-01, 0686F1000-01:FUSC1608X60N, F.Cu at (235.8, -42.5)
- added F10: 0686F1000-01, 0686F1000-01:FUSC1608X60N, F.Cu at (245.2, -34.4)
- added F11: 0686F1000-01, 0686F1000-01:FUSC1608X60N, F.Cu at (245.2, -31.7)
- added F12: 0686F1000-01, 0686F1000-01:FUSC1608X60N, F.Cu at (249.2, -42.5)
- added F13: 0686F1000-01, 0686F1000-01:FUSC1608X60N, F.Cu at (249.2, -39.8)
- added F14: 0686F1000-01, 0686F1000-01:FUSC1608X60N, F.Cu at (249.2, -37.1)
- added F15: 0686F1000-01, 0686F1000-01:FUSC1608X60N, F.Cu at (249.2, -34.4)
- added F16: 0438.250WRA, 0438.250WRA:FUSC1608X61N, F.Cu at (199.3, -20.0)
- added F17: 0438.250WRA, 0438.250WRA:FUSC1608X61N, F.Cu at (183.8, -15.0)
- added F18: 0438.250WRA, 0438.250WRA:FUSC1608X61N, F.Cu at (183.8, -12.4)
- added F19: 0438.250WRA, 0438.250WRA:FUSC1608X61N, F.Cu at (183.8, -9.86)
- added F2: 0686F1000-01, 0686F1000-01:FUSC1608X60N, F.Cu at (241.2, -42.5)
- added F20: 0438.250WRA, 0438.250WRA:FUSC1608X61N, F.Cu at (183.8, -7.29)
- added F21: 0438.250WRA, 0438.250WRA:FUSC1608X61N, F.Cu at (183.8, -4.72)
- added F22: 0438.250WRA, 0438.250WRA:FUSC1608X61N, F.Cu at (187.8, -15.0)
- added F23: 0438.250WRA, 0438.250WRA:FUSC1608X61N, F.Cu at (187.8, -12.4)
- added F24: 0438.250WRA, 0438.250WRA:FUSC1608X61N, F.Cu at (187.8, -9.86)
- added F25: 0438.250WRA, 0438.250WRA:FUSC1608X61N, F.Cu at (187.8, -7.29)
- added F26: 0438.250WRA, 0438.250WRA:FUSC1608X61N, F.Cu at (187.8, -4.72)
- added F27: 0438.250WRA, 0438.250WRA:FUSC1608X61N, F.Cu at (191.8, -15.0)
- added F28: 0438.250WRA, 0438.250WRA:FUSC1608X61N, F.Cu at (191.8, -12.4)
- added F29: 0438.250WRA, 0438.250WRA:FUSC1608X61N, F.Cu at (191.8, -9.86)
- added F3: 0686F1000-01, 0686F1000-01:FUSC1608X60N, F.Cu at (241.2, -39.8)
- added F30: 0438.250WRA, 0438.250WRA:FUSC1608X61N, F.Cu at (191.8, -7.29)
- added F4: 0686F1000-01, 0686F1000-01:FUSC1608X60N, F.Cu at (241.2, -37.1)
- added F5: 0686F1000-01, 0686F1000-01:FUSC1608X60N, F.Cu at (241.2, -34.4)
- added F6: 0686F1000-01, 0686F1000-01:FUSC1608X60N, F.Cu at (241.2, -31.7)
- added F7: 0686F1000-01, 0686F1000-01:FUSC1608X60N, F.Cu at (245.2, -42.5)
- added F8: 0686F1000-01, 0686F1000-01:FUSC1608X60N, F.Cu at (245.2, -39.8)
- added F9: 0686F1000-01, 0686F1000-01:FUSC1608X60N, F.Cu at (245.2, -37.1)
Connections:
- net Net-(C1-Pad2) renamed /BQ79614_Bootstrapping/Cell 14S PIN
- R10 pad 2: Cell 2 -> Net-(F3-Pad2)
- R11 pad 2: Cell 1 -> Net-(F2-Pad2)
- R12 pad 2: Cell 0 -> Net-(F1-Pad2)
- R13 pad 2: Cell 10 -> Net-(F11-Pad2)
- R14 pad 2: Cell 9 -> Net-(F10-Pad2)
- R15 pad 2: Cell 8 -> Net-(F9-Pad2)
- R16 pad 2: Cell 7 -> Net-(F8-Pad2)
- R17 pad 2: Cell 6 -> Net-(F7-Pad2)
- R18 pad 2: Cell 5 -> Net-(F6-Pad2)
- R19 pad 2: Cell 4 -> Net-(F5-Pad2)
- R2 pad 2: Cell 10 -> Net-(F11-Pad2)
- R20 pad 2: Cell 3 -> Net-(F4-Pad2)
- R21 pad 2: Cell 2 -> Net-(F3-Pad2)
- R22 pad 2: Cell 1 -> Net-(F2-Pad2)
- R23 pad 2: Cell 0 -> Net-(F1-Pad2)
- R24 pad 2: Cell 11 -> Net-(F12-Pad2)
- R25 pad 2: Cell 12 -> Net-(F13-Pad2)
- R26 pad 2: Cell 13 -> Net-(F14-Pad2)
- R27 pad 2: Cell 14S -> Net-(F15-Pad2)
- R28 pad 2: Cell 14S -> Net-(F15-Pad2)
- R29 pad 2: Cell 13 -> Net-(F14-Pad2)
- R3 pad 2: Cell 9 -> Net-(F10-Pad2)
- R30 pad 2: Cell 12 -> Net-(F13-Pad2)
- R31 pad 2: Cell 11 -> Net-(F12-Pad2)
- R4 pad 2: Cell 8 -> Net-(F9-Pad2)
- R5 pad 2: Cell 7 -> Net-(F8-Pad2)
- R6 pad 2: Cell 6 -> Net-(F7-Pad2)
- R7 pad 2: Cell 5 -> Net-(F6-Pad2)
- R8 pad 2: Cell 4 -> Net-(F5-Pad2)
- R9 pad 2: Cell 3 -> Net-(F4-Pad2)
- TP18 pad TP: Cell 10 -> Net-(F11-Pad2)
- TP19 pad TP: Cell 9 -> Net-(F10-Pad2)
- TP20 pad TP: Cell 8 -> Net-(F9-Pad2)
- TP21 pad TP: Cell 7 -> Net-(F8-Pad2)
- TP22 pad TP: Cell 6 -> Net-(F7-Pad2)
- TP23 pad TP: Cell 5 -> Net-(F6-Pad2)
- TP24 pad TP: Cell 4 -> Net-(F5-Pad2)
- TP25 pad TP: Cell 3 -> Net-(F4-Pad2)
- TP26 pad TP: Cell 2 -> Net-(F3-Pad2)
- TP27 pad TP: Cell 1 -> Net-(F2-Pad2)
- TP28 pad TP: Cell 11 -> Net-(F12-Pad2)
- TP29 pad TP: Cell 12 -> Net-(F13-Pad2)
- TP30 pad TP: Cell 13 -> Net-(F14-Pad2)
- TP31 pad TP: Cell 14S -> Net-(F15-Pad2)

Commit message: m
Parts:
- moved C45 101.9 mm to (257.3, -56.3)
- moved D1 101.9 mm to (261.7, -57.5)
- moved FL2 101.9 mm to (246.6, -56.8)
- moved J2 101.9 mm to (249.5, -73.7)
- moved J3 101.9 mm to (266.2, -73.7)
- moved R39 101.9 mm to (253.3, -58.8)
- moved R40 101.9 mm to (253.3, -56.3)
- moved R41 101.9 mm to (239.9, -58.8)
- moved R42 101.9 mm to (239.9, -56.3)
- moved R49 101.9 mm to (239.9, -53.9)
- moved R51 101.9 mm to (235.9, -72.5)
- moved R53 101.9 mm to (235.9, -66.9)
- moved R54 101.9 mm to (235.9, -64.1)
- moved C42 101.9 mm to (257.3, -58.8)
- moved R50 101.9 mm to (235.9, -75.3)
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
Commit message: Starting Routing
Parts:
- moved TP27 217.8 mm to (129.5, 129.5)
- moved TP25 217.4 mm to (129.5, 119.4)
- moved TP26 217.3 mm to (129.5, 124.5)
- moved TP24 217.1 mm to (129.5, 114.3)
- moved F1 204.0 mm to (108.4, 116.8)
- moved F2 203.5 mm to (108.4, 111.8)
- moved F3 199.6 mm to (108.4, 109.2)
- moved R12 198.7 mm to (166.5, 134.6), turned to 180 degrees
- moved F7 196.9 mm to (108.4, 99.1)
- moved R11 196.8 mm to (166.3, 129.5), turned to 180 degrees
- moved F4 195.7 mm to (108.4, 106.7)
- moved R10 195.0 mm to (166.3, 124.5), turned to 180 degrees
- moved TP32 193.3 mm to (129.5, 134.6)
- moved F8 193.2 mm to (108.3, 96.5)
- moved R9 193.1 mm to (166.3, 119.4), turned to 180 degrees
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Connections:
- R10 pad 1: CB2 -> Net-(F3-Pad2)
- R10 pad 2: Net-(F3-Pad2) -> CB2
- R11 pad 1: CB1 -> Net-(F2-Pad2)
- R11 pad 2: Net-(F2-Pad2) -> CB1
- R2 pad 1: CB10 -> Net-(F11-Pad2)
- R2 pad 2: Net-(F11-Pad2) -> CB10
- R24 pad 1: CB11 -> Net-(F12-Pad2)
- R24 pad 2: Net-(F12-Pad2) -> CB11
- R25 pad 1: CB12 -> Net-(F13-Pad2)
- R25 pad 2: Net-(F13-Pad2) -> CB12
- R26 pad 1: CB13 -> Net-(F14-Pad2)
- R26 pad 2: Net-(F14-Pad2) -> CB13
- R27 pad 1: CB14 -> Net-(F15-Pad2)
- R27 pad 2: Net-(F15-Pad2) -> CB14
- R28 pad 1: VC14 -> Net-(F15-Pad2)
- R28 pad 2: Net-(F15-Pad2) -> VC14
- R3 pad 1: CB9 -> Net-(F10-Pad2)
- R3 pad 2: Net-(F10-Pad2) -> CB9
- R4 pad 1: CB8 -> Net-(F9-Pad2)
- R4 pad 2: Net-(F9-Pad2) -> CB8
- R5 pad 1: CB7 -> Net-(F8-Pad2)
- R5 pad 2: Net-(F8-Pad2) -> CB7
- R6 pad 1: CB6 -> Net-(F7-Pad2)
- R6 pad 2: Net-(F7-Pad2) -> CB6
- R7 pad 1: CB5 -> Net-(F6-Pad2)
- R7 pad 2: Net-(F6-Pad2) -> CB5
- R8 pad 1: CB4 -> Net-(F5-Pad2)
- R8 pad 2: Net-(F5-Pad2) -> CB4
- R9 pad 1: CB3 -> Net-(F4-Pad2)
- R9 pad 2: Net-(F4-Pad2) -> CB3
Other:
- copper layers 2 -> 4
