File: DaughterBoard/Project63_BMS_DaughterBoard.kicad_pcb (KiCad board)
At the start: 4 copper layers, 193 parts, among them J1 705550019, J2 705510038, J2 PEC03SAAN, J3 705510038, J3 PEC02SAAN, J4 PEC02SAAN, Q1 ZXTN4004KTC, U1 BQ79614PAPRQ1

Commit message: C:/Program Files/Git/
Parts:
- R36: value 1.00K -> 1k
- moved TP17 1.05 mm to (179.5, -69.0)
- moved TP10 0.72 mm to (148.0, -70.1)
- moved J2 0.58 mm to (288.5, -96.0)
Connections:
- C40 pad 1: /COMML/GND -> AVSS
- C41 pad 1: /COMML/GND -> AVSS
- C42 pad 1: /COMML/GND -> AVSS
- C42 pad 2: COMLN -> COMHN
- C45 pad 1: /COMML/GND -> AVSS
- C45 pad 2: COMLP -> COMHP
- D1 pad 3: /COMML/GND -> AVSS
- D2 pad 3: /COMML/GND -> AVSS
- J2 pad 1: /COMML/ISO_COMML_N -> ISO_COMML_N
- J2 pad 2: /COMML/ISO_COMML_P -> ISO_COMML_P
- J3 pad 1: /COMML/ISO_COMML_N -> ISO_COMMH_N
- J3 pad 2: /COMML/ISO_COMML_P -> ISO_COMMH_P
- R37 pad 1: /COMML/COMML_N_OPT -> COMML_N_OPT
- R38 pad 1: /COMML/COMML_P_OPT -> COMML_P_OPT
- R39 pad 1: /COMML/COMML_N_OPT -> COMMH_N_OPT
- R40 pad 1: /COMML/COMML_P_OPT -> COMMH_P_OPT
- R41 pad 1: COMLP -> COMHP
- R42 pad 1: COMLN -> COMHN
- R43 pad 2: /COMML/ISO_COMML_P -> ISO_COMML_P
- R44 pad 2: /COMML/ISO_COMML_N -> ISO_COMML_N
- R45 pad 1: /COMML/COMML_P_OPT -> COMML_P_OPT
- R46 pad 1: /COMML/COMML_N_OPT -> COMML_N_OPT
- R49 pad 1: COMLN -> COMHN
- R49 pad 2: COMLP -> COMHP
- R50 pad 2: /COMML/ISO_COMML_P -> ISO_COMMH_P
- R51 pad 2: /COMML/ISO_COMML_N -> ISO_COMMH_N
- R54 pad 1: /COMML/COMML_P_OPT -> COMMH_P_OPT
- R55 pad 1: /COMML/COMML_N_OPT -> COMMH_N_OPT
- TP32 pad TP: Cell 0 -> Net-(F1-Pad2)

Commit message: Layout continued. Fixed Footprint and most 3d model
Parts:
- removed the C42 at (280.4, -95.5)
- removed the J2 at (288.5, -96.0)
- removed the J3 at (290.1, -111.8)
- removed J4: PEC02SAAN, PEC02SAAN:CONN_PxC02S_SUL
- removed the R39 at (280.3, -113.5)
- removed the R40 at (280.3, -110.8)
- removed the R41 at (280.3, -108.0)
- removed the R42 at (280.3, -105.2)
- added C46: 2200pF, 1206J2K00222KXR (1):CAPC3216X160N, F.Cu at (244.4, 65.2)
- added C47: 2200pF, 1206J2K00222KXR (1):CAPC3216X160N, F.Cu at (239.8, 65.2)
- C39: footprint GCM31MR72A224KA3L:G-31_MUR -> GCM31MR72A224KA37L:G-31_MUR-L
- C40, C41: footprint CL10B221JB8NNNC:CAP_CL10_SAM -> CL10B221JB8NNNC:CAP_CL10_SAM-L
- D1, D2: footprint PESD1CAN,215:SOT23_PESD1_NEX -> PESD1CAN_215:SOT23_PESD1_NEX
- FL1, FL2: footprint 744242471:744242471 -> KiCad:744242471
- J2, J3: footprint 70551-0038:CONN_70551-xxxx_04_MOL -> 0705510038:CONN_70551-xxxx_04_MOL
- Q1: footprint ZXTN4004KTC:ZXTN4004KTC -> LIB_ZXTN4004KTC:ZXTN4004KTC
- R32: footprint CRCW2010100RFKEF:RES_CRCW_2010 -> CRCW2010100RFKEF:RES_CRCW_2010-L
- R34, R35: footprint CRCW060351R0JNEA:RC0603N_VIS -> CRCW060351R0JNEA:RC0603N_VIS-L
- R36: footprint ERA-3AEB101V:RC0603N_PAN -> ERJ-3EKF1001V:RC0603N_PAN-L
- R39, R40: footprint RC0603JR-070RL:RC0603N_YAG -> RC0603JR-070RL:RC0603N_YAG-L
- R49: value 1.00K -> 1K; footprint ERA-3AEB101V:RC0603N_PAN -> ERJ-3EKF1001V:RC0603N_PAN
- moved R44 257.4 mm to (243.7, 140.7), turned to -90 degrees
- moved R43 246.3 mm to (241.2, 140.7), turned to -90 degrees
- moved R23 243.4 mm to (144.8, 132.1)
- moved R47 240.2 mm to (236.8, 130.3), turned to -90 degrees
- moved C43 240.1 mm to (244.6, 120.9), turned to 90 degrees
- moved Q1 239.7 mm to (210.8, 73.7)
- moved C44 238.0 mm to (239.5, 120.9), turned to 90 degrees
- moved R22 237.2 mm to (144.8, 127.0), turned to 180 degrees
- moved FL1 236.7 mm to (242.4, 130.4), turned to 90 degrees
- moved R48 235.6 mm to (248.1, 130.4), turned to -90 degrees
- moved R21 231.0 mm to (144.8, 121.9), turned to 180 degrees
- moved R45 228.4 mm to (239.5, 113.3), turned to -90 degrees
- moved J2 225.2 mm to (243.7, 148.6)
- moved R20 224.9 mm to (144.8, 116.8), turned to 180 degrees
- moved R46 224.8 mm to (244.6, 113.3), turned to -90 degrees
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Connections:
- J3 pad 1: ISO_COMMH_N -> unconnected-(J3-Pad1)
- J3 pad 2: ISO_COMMH_P -> unconnected-(J3-Pad2)
- J3 pad 3: unconnected-(J3-Pad3) -> ISO_COMMH_N
- J3 pad 4: unconnected-(J3-Pad4) -> ISO_COMMH_P
- R23 pad 1: VC0 -> Net-(F1-Pad2)
- R23 pad 2: Net-(F1-Pad2) -> VC0

Commit message: tracing left
Parts:
- C42, C45: footprint CL10B221JB8NNNC:CAP_CL10_SAM -> CL10B221JB8NNNC:CAP_CL10_SAM-L
- D1, D2: footprint PESD1CAN_215:SOT23_PESD1_NEX -> PESD1CAN,215:SOT23_PESD1_NEX
- Q1: footprint LIB_ZXTN4004KTC:ZXTN4004KTC -> ZXTN4004KTC:ZXTN4004KTC
- R1: value 30 Ohm -> 30; footprint ERJ-3EKF30R0V:RC0603N_PAN -> ERJ-3EKF30R0V:RC0603N_PAN-L
- R10, R4, R5: value 7.5 ohm -> 7.5
- R11, R12, R2, R24, R25, R26, R27, R3, R6, R7, R8, R9: value 7.5 Ohm -> 7.5
- R13, R14, R15, R16, R17, R18, R19, R20, R21, R22, R23, R28, R29, R30, R31: value 100 Ohm -> 100
- R32: value 100 -> 100
- R33: value 200 -> 200; footprint CRCW2010200RFKEF:RC2010N_VIS -> CRCW2010200RFKEF:RC2010N_VIS-L
- R34, R35: value 51 -> 51
- R37, R38: value 0 -> 0; footprint RC0603JR-070RL:RC0603N_YAG -> RC0603JR-070RL:RC0603N_YAG-L
- R39, R40: value 0 -> 0
- R41, R42: value 51 -> 51; footprint CRCW060351R0JNEA:RC0603N_VIS -> CRCW060351R0JNEA:RC0603N_VIS-L
- R43, R44, R45, R46, R47, R48, R50, R51, R52, R53, R54, R55: value 0 -> 0; footprint CRCW08050000Z0EAHP:RES_CRCW_0805_VIS -> CRCW08050000Z0EAHP:RES_CRCW_0805_VIS-L
- R49: value 1K -> 1k; footprint ERJ-3EKF1001V:RC0603N_PAN -> ERJ-3EKF1001V:RC0603N_PAN-L
- TP1, TP10, TP11, TP12, TP13, TP14, TP18, TP19, TP2, TP20, TP21, TP22, TP23, TP24, TP25, TP26, TP27, TP28, TP29, TP3, TP30, TP31, TP4, TP5, TP6, TP7, TP8, TP9: footprint TP5012:TP_5012 -> 5012:TP_5012

Commit message: Connectors
Parts:
- removed J2, J3: 705510038, 0705510038:CONN_70551-xxxx_04_MOL
- removed the TP1 at (168.9, -90.2)
- removed the TP10 at (174.0, -75.0)
- removed the TP11 at (174.0, -70.0)
- removed the TP12 at (174.0, -64.9)
- removed the TP13 at (179.1, -90.2)
- removed the TP14 at (179.1, -85.1)
- removed TP15, TP16, TP17: ~, TestPoint:TestPoint_Keystone_5010-5014_Multipurpose
- removed the TP2 at (168.9, -85.1)
- removed the TP3 at (168.9, -80.0)
- removed the TP4 at (168.9, -75.0)
- removed the TP5 at (168.9, -70.0)
- removed the TP6 at (168.9, -64.9)
- removed the TP7 at (174.0, -90.2)
- removed the TP8 at (174.0, -85.1)
- removed the TP9 at (174.0, -80.0)
- added J4: 1-794106-0, 1-794106-0:CON20_2X10_P4.14MM_RAMNL_TYC, F.Cu at (85.1, 117.5)
- added J5: 430450200, 0430450200:CON_430450200_MOL, F.Cu at (215.2, 36.0)
- D1, D2: footprint PESD1CAN,215:SOT23_PESD1_NEX -> PESD1CAN_215:SOT23_PESD1_NEX
- J1: value 705550019 -> 430450200; footprint 705550019:CONN_705550019_MOL -> 0430450200:CON_430450200_MOL
- moved J1 130.8 mm to (215.2, 156.2), turned to 0 degrees
- moved R40 26.3 mm to (218.3, 78.2)
- moved C42 26.3 mm to (213.4, 91.3)
- moved C43 26.3 mm to (218.5, 124.0)
- moved C44 26.3 mm to (213.4, 124.0)
- moved C46 26.3 mm to (218.2, 68.2)
- moved D1 26.3 mm to (215.9, 83.4)
- moved D2 26.3 mm to (216.1, 107.4)
- moved FL2 26.3 mm to (216.0, 58.6)
- moved R34 26.3 mm to (213.4, 103.6)
- moved R35 26.3 mm to (218.5, 103.6)
- moved R37 26.3 mm to (218.5, 112.1)
- moved R38 26.3 mm to (213.4, 112.1)
- moved R41 26.3 mm to (219.0, 87.1)
- moved R45 26.3 mm to (213.4, 116.3)
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Connections:
- J1 pad 1: Cell 0 -> ISO_COMML_N
- J1 pad 2: Cell 14 -> ISO_COMML_P

Commit message: Test
Parts:
- moved C4 217.8 mm to (289.6, -22.2), turned to 90 degrees
- moved C30 206.8 mm to (278.9, -22.0), turned to -90 degrees
- moved C29 206.1 mm to (278.3, -18.7), turned to 180 degrees
- moved C2 203.0 mm to (278.9, -25.7), turned to -90 degrees
- moved C8 202.0 mm to (278.3, -30.1), turned to 180 degrees
- moved C28 201.4 mm to (273.6, -15.0), turned to 180 degrees
- moved C27 198.7 mm to (271.4, -13.3), turned to 180 degrees
- moved C26 196.4 mm to (270.4, -14.9), turned to 180 degrees
- moved C25 193.6 mm to (268.2, -13.2), turned to 180 degrees
- moved C24 191.1 mm to (267.2, -15.0)
- moved C23 188.6 mm to (265.2, -13.2), turned to 180 degrees
- moved C22 186.2 mm to (263.9, -15.0), turned to 180 degrees
- moved C21 180.4 mm to (259.9, -17.8), turned to 90 degrees
- moved C20 127.7 mm to (203.3, -10.3), turned to 90 degrees
- moved C38 127.4 mm to (205.1, -11.3), turned to 90 degrees
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
Commit message: test
Parts:
- removed TP10, TP12, TP13, TP8: 5012, 5012:TP_5012
- D1, D2: footprint PESD1CAN_215:SOT23_PESD1_NEX -> PESD1CAN,215:SOT23_PESD1_NEX
- moved C17 191.8 mm to (173.9, 104.5), turned to 180 degrees
- moved C13 187.4 mm to (168.9, 104.5), turned to 180 degrees
- moved C15 183.3 mm to (171.4, 104.5), turned to 180 degrees
- moved C11 178.8 mm to (166.4, 104.5), turned to 180 degrees
- moved C9 175.8 mm to (159.5, 98.3), turned to 90 degrees
- moved C36 173.0 mm to (161.0, 94.3), turned to 90 degrees
- moved TP6 167.8 mm to (186.0, 122.0)
- moved C18 166.5 mm to (235.3, -13.0), turned to 180 degrees
- moved C33 165.9 mm to (159.5, 95.8), turned to 90 degrees
- moved C16 160.8 mm to (231.9, -13.0), turned to 180 degrees
- moved TP5 160.3 mm to (152.0, 89.0)
- moved TP9 160.0 mm to (190.5, 76.0)
- moved TP7 157.2 mm to (186.0, 107.0)
- moved C14 156.4 mm to (228.6, -13.0), turned to 180 degrees
- moved C21 153.4 mm to (165.4, 103.0), turned to 180 degrees
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Connections:
- C3 pad 2: REFHP -> REFHF
- U1 pad 36: AVSS -> REFHP
- U1 pad 37: REFHP -> REFHF
- U1 pad EPAD: unconnected-(U1-PadEPAD) -> AVSS

Commit message: layout
Parts:
- C10, C11, C12, C13, C14, C15, C16, C17, C18, C31, C32, C33, C34, C9: moved to B.Cu
- moved C20 136.6 mm to (161.5, 100.5), turned to 180 degrees
- moved C22 133.8 mm to (164.0, 100.5), turned to 180 degrees
- moved C35 133.7 mm to (157.5, 90.0), turned to 90 degrees
- moved C37 133.6 mm to (157.5, 92.4), turned to 90 degrees
- moved C24 131.1 mm to (166.6, 100.5), turned to 180 degrees
- moved C16 129.8 mm to (168.7, 100.5), turned to 0 degrees
- moved C14 129.4 mm to (166.4, 100.5), turned to 0 degrees
- moved C12 128.9 mm to (163.9, 100.5), turned to 0 degrees
- moved C26 128.9 mm to (169.1, 100.5), turned to 180 degrees
- moved C10 128.6 mm to (161.5, 100.5), turned to 0 degrees
- moved C18 127.5 mm to (171.6, 97.5), turned to 0 degrees
- moved C28 123.8 mm to (172.1, 97.5), turned to 180 degrees
- moved C34 121.4 mm to (157.5, 91.8), turned to 90 degrees
- moved C32 117.5 mm to (157.5, 89.3), turned to 90 degrees
- moved C30 40.9 mm to (181.5, 5.00), turned to -90 degrees
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
Commit message: done
Parts:
- C10, C11, C12, C13, C14, C15, C16, C17, C18, C31, C32, C33, C34, C9: moved to F.Cu
- moved C30 88.5 mm to (177.0, 93.4)
- moved C29 88.2 mm to (177.0, 95.9)
- moved C19 87.9 mm to (175.5, 93.4)
- moved C3 84.8 mm to (177.0, 90.9), turned to -90 degrees
- moved C4 82.3 mm to (177.0, 88.1)
- moved C7 78.6 mm to (169.5, 81.9), turned to 0 degrees
- moved C5 77.6 mm to (166.9, 81.9), turned to 180 degrees
- moved C18 5.95 mm to (177.4, 99.0), turned to 180 degrees
- moved C28 5.41 mm to (176.6, 100.5)
- moved C20 4.62 mm to (156.9, 100.5)
- moved C10 4.38 mm to (157.4, 99.0), turned to 180 degrees
- moved C17 4.26 mm to (174.9, 99.0), turned to 180 degrees
- moved C27 4.16 mm to (174.3, 100.5)
- moved C16 3.94 mm to (172.4, 99.0), turned to 180 degrees
- moved C21 3.92 mm to (159.4, 100.5)
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