File: DaughterBoard/BQ79614_bootstrapping.kicad_sch (KiCad schematic)
At the start: 10 parts, among them U1 BQ79614PAPRQ1

Commit message: Daughter Update
Connections:
- net GND_AVSS is gone; now on net GND: C1.1, C4.1
- net GND_CVSS is gone; now on net GND: C2.1, C5.1, C6.1, C8.1
- net GND_DVSS is gone; now on net GND: C7.1
- net GND_REFHM is gone; now on net GND: C3.1
- net PWR renamed Cell 14S

Commit message: 11/9/2024
Connections:
- net GND: no longer U1.EPAD
- no-connect marks 16 -> 17

Commit message: only fuses left
Connections:
- net Cell 14S PIN: now reaches C1.2, R1.1, U1.1
Changed lines of the file:
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@@
+		)
+	)
+	(label "Cell 14S PIN"
+		(at 77.47 49.53 0)
+		(fields_autoplaced yes)
+		(effects
+			(font
+				(size 1.27 1.27)
+			)
+			(justify left bottom)
 		)
 	)

Commit message: C:/Program Files/Git/
Parts:
- C6: Manufacturer Part Number (none) -> C2012X7R1A475M125AC
- U1: Manufacturer Part Number (none) -> BQ79614PAPRQ1
Changed lines of the file:
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@@
 			)
 		)
-		(property "Manufacturer Part Number" ""
+		(property "Manufacturer Part Number" "BQ79614PAPRQ1"
 			(at 95.25 49.53 0)
 			(effects
@@
 			(at 248.92 143.51 0)
 			(effects
+				(font
+					(size 1.27 1.27)
+				)
+				(hide yes)
+			)
+		)
+		(property "Manufacturer Part Number" "C2012X7R1A475M125AC"
+			(at 248.92 143.51 0)
+			(effects
