File: DaughterBoard/BQ79614_bootstrapping.kicad_sch (KiCad schematic)
At the start: 10 parts, among them U1 BQ79614PAPRQ1

Commit message: tracing left
Parts:
- R1: value 30 Ohm -> 30; footprint ERJ-3EKF30R0V:RC0603N_PAN -> ERJ-3EKF30R0V:RC0603N_PAN-L
Changed lines of the file:
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@@
 			)
 		)
-		(property "Datasheet" ""
+		(property "Datasheet" "https://content.kemet.com/datasheets/KEM_C1023_X7R_AUTO_SMD.pdf"
 			(at 226.822 92.202 0)
 			(effects
@@
 			)
 		)
-		(property "Datasheet" ""
+		(property "Datasheet" "https://search.murata.co.jp/Ceramy/image/img/A01X/G101/ENG/GCM155R71A104KA55-01.pdf"
 			(at 211.582 110.49 0)
 			(effects
@@
 			)
 		)
-		(property "Datasheet" ""
+		(property "Datasheet" "https://www.ti.com/lit/ds/symlink/bq79612-q1.pdf"
 			(at 87.376 42.418 0)
 			(effects
@@
 			)
 		)
-		(property "Datasheet" ""
+		(property "Datasheet" "https://content.kemet.com/datasheets/KEM_C1023_X7R_AUTO_SMD.pdf"
 			(at 237.49 125.984 0)
 			(effects
@@
 			)
 		)
-		(property "Datasheet" ""
+		(property "Datasheet" "https://search.murata.co.jp/Ceramy/image/img/A01X/G101/ENG/GCM188R72A103KA37-01.pdf"
 			(at 68.58 59.69 0)
 			(effects
@@
 			)
 		)
-		(property "Value" "30 Ohm"
+		(property "Value" "30 "
 			(at 57.15 45.72 0)
 			(effects
@@
 			)
 		)
-		(property "Footprint" "ERJ-3EKF30R0V:RC0603N_PAN"
+		(property "Footprint" "ERJ-3EKF30R0V:RC0603N_PAN-L"
 			(at 50.546 54.102 0)
 			(effects
@@
 			)
 		)
-		(property "Datasheet" ""
+		(property "Datasheet" "https://industrial.panasonic.com/cdbs/www-data/pdf/RDA0000/AOA0000C304.pdf"
 			(at 50.292 56.134 0)
 			(effects
@@
 			)
 		)
-		(property "Datasheet" ""
+		(property "Datasheet" "https://search.murata.co.jp/Ceramy/image/img/A01X/G101/ENG/GCM155R71A104KA55-01.pdf"
 			(at 258.318 108.712 0)
 			(effects
@@
 			)
 		)
-		(property "Datasheet" ""
+		(property "Datasheet" "https://content.kemet.com/datasheets/KEM_C1023_X7R_AUTO_SMD.pdf"
 			(at 258.826 87.884 0)
 			(effects
@@
 			)
 		)
-		(property "Datasheet" ""
+		(property "Datasheet" "https://content.kemet.com/datasheets/KEM_C1023_X7R_AUTO_SMD.pdf"
 			(at 214.63 146.812 0)
 			(effects
@@
 			)
 		)
-		(property "Datasheet" ""
+		(property "Datasheet" "https://product.tdk.com/system/files/dam/doc/product/capacitor/ceramic/mlcc/catalog/mlcc_commercial_general_en.pdf"
 			(at 244.602 143.764 0)
 			(effects

Commit message: Test
Connections:
- net GND: now also U1.EPAD
- no-connect marks 17 -> 16
Changed lines of the file:
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@@
 	)
 	(no_connect
-		(at 135.89 49.53)
-	)
-	(no_connect
 		(at 135.89 80.01)
 	)
@@
 	(wire
 		(pts
+			(xy 135.89 49.53) (xy 146.05 49.53)
+		)
+		(stroke
+			(width 0)
+			(type default)
+		)
+	)
+	(wire
+		(pts
 			(xy 90.17 80.01) (xy 95.25 80.01)
 		)
@@
 					(unit 1)
 				)
+			)
+		)
+	)
+	(symbol
+		(lib_id "power:GND")
+		(at 146.05 49.53 0)
+		(unit 1)
+		(exclude_from_sim no)
+		(in_bom yes)
+		(on_board yes)
+		(dnp no)
+		(fields_autoplaced yes)
+		(property "Reference" "#PWR014"
+			(at 146.05 55.88 0)
+			(effects
+				(font
+					(size 1.27 1.27)
+				)
+				(hide yes)
+			)
+		)
+		(property "Value" "GND"
+			(at 146.05 54.61 0)
+			(effects
+				(font
+					(size 1.27 1.27)
+				)
+			)
+		)
+		(property "Footprint" ""
+			(at 146.05 49.53 0)
+			(effects
+				(font
+					(size 1.27 1.27)
+				)
+				(hide yes)
+			)
+		)
+		(property "Datasheet" ""
+			(at 146.05 49.53 0)
+			(effects
+				(font
+					(size 1.27 1.27)
+				)
+				(hide yes)
+			)
+		)
+		(property "Description" "Power symbol creates a global label with name \"GND\" , ground"
+			(at 146.05 49.53 0)
+			(effects
+				(font
+					(size 1.27 1.27)
+				)
+				(hide yes)
+			)
+		)
+		(pin "1"
+		)
+		(instances
+			(project "Project63_BMS_DaughterBoard"
+				(path "/325b096d-8e4c-4cdc-b4c5-634ea5e73c60/8ffa0956-e90f-44b3-af43-d8470a47be31"
+					(reference "#PWR014")
+					(unit 1)
+				)

Commit message: test
Connections:
- net GND: no longer U1.36
- net REFHP: now also U1.36; no longer C3.2, U1.37
- new net REFHF: C3.2, U1.37
Changed lines of the file:
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@@
+		)
+	)
+	(global_label "REFHP"
+		(shape input)
+		(at 140.97 123.19 0)
+		(fields_autoplaced yes)
+		(effects
+			(font
+				(size 1.27 1.27)
+			)
+			(justify left)
+		)
+		(property "Intersheetrefs" "${INTERSHEET_REFS}"
+			(at 150.0633 123.19 0)
+			(effects
+				(font
+					(size 1.27 1.27)
+				)
+				(justify left)
+				(hide yes)
+			)
+		)
+	)
+	(global_label "VC3"
+		(shape input)
+		(at 90.17 120.65 180)
+		(fields_autoplaced yes)
+		(effects
+			(font
+				(size 1.27 1.27)
+			)
+			(justify right)
+		)
+		(property "Intersheetrefs" "${INTERSHEET_REFS}"
+			(at 83.6167 120.65 0)
+			(effects
+				(font
+					(size 1.27 1.27)
+				)
+				(justify right)
+				(hide yes)
+			)
+		)
+	)
+	(global_label "CB3"
+		(shape input)
+		(at 90.17 118.11 180)
+		(fields_autoplaced yes)
+		(effects
+			(font
+				(size 1.27 1.27)
+			)
+			(justify right)
+		)
+		(property "Intersheetrefs" "${INTERSHEET_REFS}"
+			(at 83.4353 118.11 0)
+			(effects
+				(font
+					(size 1.27 1.27)
+				)
+				(justify right)
+				(hide yes)
+			)
+		)
+	)
+	(global_label "VC1"
+		(shape input)
+		(at 194.31 130.81 0)
+		(fields_autoplaced yes)
+		(effects
+			(font
+				(size 1.27 1.27)
+			)
+			(justify left)
+		)
+		(property "Intersheetrefs" "${INTERSHEET_REFS}"
+			(at 200.8633 130.81 0)
+			(effects
+				(font
+					(size 1.27 1.27)
+				)
+				(justify left)
+				(hide yes)
+			)
+		)
+	)
+	(global_label "VC9"
+		(shape input)
+		(at 90.17 90.17 180)
+		(fields_autoplaced yes)
+		(effects
+			(font
+				(size 1.27 1.27)
+			)
+			(justify right)
+		)
+		(property "Intersheetrefs" "${INTERSHEET_REFS}"
+			(at 83.6167 90.17 0)
+			(effects
+				(font
+					(size 1.27 1.27)
+				)
+				(justify right)
+				(hide yes)
+			)
+		)
+	)
+	(global_label "CB2"
+		(shape input)
+		(at 90.17 123.19 180)
+		(fields_autoplaced yes)
+		(effects
+			(font
+				(size 1.27 1.27)
+			)
+			(justify right)
+		)
+		(property "Intersheetrefs" "${INTERSHEET_REFS}"
+			(at 83.4353 123.19 0)
+			(effects
+				(font
+					(size 1.27 1.27)
+				)
+				(justify right)
+				(hide yes)
+			)
+		)
+	)
+	(global_label "CB4"
+		(shape input)
+		(at 90.17 113.03 180)
+		(fields_autoplaced yes)
+		(effects
+			(font
+				(size 1.27 1.27)
+			)
+			(justify right)
+		)
+		(property "Intersheetrefs" "${INTERSHEET_REFS}"
+			(at 83.4353 113.03 0)
+			(effects
+				(font
+					(size 1.27 1.27)
+				)
+				(justify right)
+				(hide yes)
+			)
+		)
+	)
+	(global_label "CB0"
+		(shape input)
+		(at 194.31 128.27 0)
+		(fields_autoplaced yes)
+		(effects
+			(font
+				(size 1.27 1.27)
+			)
+			(justify left)
+		)
+		(property "Intersheetrefs" "${INTERSHEET_REFS}"
+			(at 201.0447 128.27 0)
+			(effects
+				(font
+					(size 1.27 1.27)
+				)
+				(justify left)
+				(hide yes)
+			)
 		)
 	)
 	(global_label "REFHM"
 		(shape input)
-		(at 140.97 123.19 0)
-		(fields_autoplaced yes)
-		(effects
-			(font
-				(size 1.27 1.27)
-			)
-			(justify left)
-		)
-		(property "Intersheetrefs" "${INTERSHEET_REFS}"
-			(at 150.2447 123.19 0)
-			(effects
-				(font
-					(size 1.27 1.27)
-				)
-				(justify left)
-				(hide yes)
-			)
-		)
-	)
-	(global_label "VC3"
-		(shape input)
-		(at 90.17 120.65 180)
-		(fields_autoplaced yes)
-		(effects
-			(font
-				(size 1.27 1.27)
-			)
-			(justify right)
-		)
-		(property "Intersheetrefs" "${INTERSHEET_REFS}"
-			(at 83.6167 120.65 0)
-			(effects
-				(font
-					(size 1.27 1.27)
-				)
-				(justify right)
-				(hide yes)
-			)
-		)
-	)
-	(global_label "CB3"
-		(shape input)
-		(at 90.17 118.11 180)
-		(fields_autoplaced yes)
-		(effects
-			(font
-				(size 1.27 1.27)
-			)
-			(justify right)
-		)
-		(property "Intersheetrefs" "${INTERSHEET_REFS}"
-			(at 83.4353 118.11 0)
-			(effects
-				(font
-					(size 1.27 1.27)
-				)
-				(justify right)
-				(hide yes)
-			)
-		)
-	)
-	(global_label "VC1"
-		(shape input)
-		(at 194.31 130.81 0)
-		(fields_autoplaced yes)
-		(effects
-			(font
-				(size 1.27 1.27)
-			)
-			(justify left)
-		)
-		(property "Intersheetrefs" "${INTERSHEET_REFS}"
-			(at 200.8633 130.81 0)
-			(effects
-				(font
-					(size 1.27 1.27)
-				)
-				(justify left)
-				(hide yes)
-			)
-		)
-	)
-	(global_label "VC9"
-		(shape input)
-		(at 90.17 90.17 180)
-		(fields_autoplaced yes)
-		(effects
-			(font
-				(size 1.27 1.27)
-			)
-			(justify right)
-		)
-		(property "Intersheetrefs" "${INTERSHEET_REFS}"
-			(at 83.6167 90.17 0)
-			(effects
-				(font
-					(size 1.27 1.27)
-				)
-				(justify right)
-				(hide yes)
-			)
-		)
-	)
-	(global_label "CB2"
-		(shape input)
-		(at 90.17 123.19 180)
-		(fields_autoplaced yes)
-		(effects
-			(font
-				(size 1.27 1.27)
-			)
-			(justify right)
-		)
-		(property "Intersheetrefs" "${INTERSHEET_REFS}"
-			(at 83.4353 123.19 0)
-			(effects
-				(font
-					(size 1.27 1.27)
-				)
-				(justify right)
-				(hide yes)
-			)
-		)
-	)
-	(global_label "CB4"
-		(shape input)
-		(at 90.17 113.03 180)
-		(fields_autoplaced yes)
-		(effects
-			(font
-				(size 1.27 1.27)
-			)
-			(justify right)
-		)
-		(property "Intersheetrefs" "${INTERSHEET_REFS}"
-			(at 83.4353 113.03 0)
-			(effects
-				(font
-					(size 1.27 1.27)
-				)
-				(justify right)
-				(hide yes)
-			)
-		)
-	)
-	(global_label "CB0"
-		(shape input)
-		(at 194.31 128.27 0)
-		(fields_autoplaced yes)
-		(effects
-			(font
-				(size 1.27 1.27)
-			)
-			(justify left)
-		)
-		(property "Intersheetrefs" "${INTERSHEET_REFS}"
-			(at 201.0447 128.27 0)
-			(effects
-				(font
-					(size 1.27 1.27)
-				)
-				(justify left)
-				(hide yes)
-			)
-		)
-	)
-	(global_label "REFHM"
-		(shape input)
 		(at 226.06 147.32 0)
 		(fields_autoplaced yes)
@@
 		)
 	)
-	(global_label "REFHP"
+	(global_label "REFHF"
 		(shape input)
 		(at 231.14 139.7 0)
@@
 		)
 		(property "Intersheetrefs" "${INTERSHEET_REFS}"
-			(at 240.2333 139.7 0)
-			(effects
-				(font
+			(at 240.0519 139.7 0)
+			(effects
+				(font

Commit message: Initial Routing
Connections:
- net REFHF is gone; now on net REFHP: C3.2, U1.37
- net GND: now also U1.36
- net REFHP: no longer U1.36
- net Cell 14S renamed BAT

Commit message: Routing Update 3
Parts:
- added NT1, NT2, NT3, NT4: NetTie_2, symbol Device:NetTie_2
- R1: value 30 -> 30
Connections:
- net GND: now also NT1.1, NT1.2, NT2.1, NT3.1, NT4.1; no longer C2.1, C3.1, C5.1, C6.1, C7.1, C8.1, U1.36, U1.46, U1.50
- net NFAULT: now reaches U1.62
- new net GND_CVSS: C2.1, C5.1, C6.1, C8.1, NT2.2, U1.46
- new net GND_DVSS: C7.1, NT3.2, U1.50
- new net GND_REFHM: C3.1, NT4.2, U1.36
- no-connect marks 16 -> 15

Commit message: Silkscreen edits
Connections:
- net Cell 14S PIN: now also U1.2, U1.3, U1.4, U1.5
- no-connect marks 15 -> 11
Changed lines of the file:
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@@
+	)
+	(junction
+		(at 92.71 49.53)
+		(diameter 0)
+		(color 0 0 0 0)
 	)
 	(junction
@@
 	)
 	(junction
+		(at 93.98 49.53)
+		(diameter 0)
+		(color 0 0 0 0)
+	)
+	(junction
 		(at 264.16 107.95)
 		(diameter 0)
@@
 	)
 	(junction
+		(at 95.25 49.53)
+		(diameter 0)
+		(color 0 0 0 0)
+	)
+	(junction
 		(at 248.92 143.51)
 		(diameter 0)
@@
 	)
 	(junction
+		(at 91.44 49.53)
+		(diameter 0)
+		(color 0 0 0 0)
+	)
+	(junction
 		(at 223.52 118.11)
 		(diameter 0)
@@
 		(diameter 0)
 		(color 0 0 0 0)
-	)
-	(no_connect
-		(at 95.25 54.61)
 	)
 	(no_connect
@@
 	)
 	(no_connect
-		(at 95.25 52.07)
-	)
-	(no_connect
 		(at 135.89 64.77)
 	)
@@
 		(at 135.89 59.69)
 	)
-	(no_connect
-		(at 95.25 59.69)
-	)
-	(no_connect
-		(at 95.25 57.15)
-	)
 	(wire
 		(pts
@@
 	(wire
 		(pts
-			(xy 68.58 49.53) (xy 95.25 49.53)
+			(xy 68.58 49.53) (xy 91.44 49.53)
 		)
 		(stroke
@@
 	(wire
 		(pts
+			(xy 91.44 59.69) (xy 91.44 49.53)
+		)
+		(stroke
+			(width 0)
+			(type default)
+		)
+	)
+	(wire
+		(pts
 			(xy 269.24 107.95) (xy 264.16 107.95)
 		)
@@
 	(wire
 		(pts
+			(xy 92.71 49.53) (xy 93.98 49.53)
+		)
+		(stroke
+			(width 0)
+			(type default)
+		)
+	)
+	(wire
+		(pts
 			(xy 167.64 76.2) (xy 167.64 72.39)
 		)
@@
 	(wire
 		(pts
+			(xy 92.71 57.15) (xy 92.71 49.53)
+		)
+		(stroke
+			(width 0)
+			(type default)
+		)
+	)
+	(wire
+		(pts
 			(xy 144.78 49.53) (xy 135.89 49.53)
 		)
@@
 	(wire
 		(pts
+			(xy 93.98 54.61) (xy 93.98 49.53)
+		)
+		(stroke
+			(width 0)
+			(type default)
+		)
+	)
+	(wire
+		(pts
 			(xy 135.89 97.79) (xy 140.97 97.79)
 		)
@@
 	(wire
 		(pts
+			(xy 95.25 59.69) (xy 91.44 59.69)
+		)
+		(stroke
+			(width 0)
+			(type default)
+		)
+	)
+	(wire
+		(pts
+			(xy 95.25 57.15) (xy 92.71 57.15)
+		)
+		(stroke
+			(width 0)
+			(type default)
+		)
+	)
+	(wire
+		(pts
+			(xy 93.98 49.53) (xy 95.25 49.53)
+		)
+		(stroke
+			(width 0)
+			(type default)
+		)
+	)
+	(wire
+		(pts
 			(xy 135.89 87.63) (xy 140.97 87.63)
 		)
@@
 	(wire
 		(pts
+			(xy 91.44 49.53) (xy 92.71 49.53)
+		)
+		(stroke
+			(width 0)
+			(type default)
+		)
+	)
+	(wire
+		(pts
 			(xy 149.86 64.77) (xy 167.64 64.77)
 		)
@@
 	(wire
 		(pts
+			(xy 95.25 49.53) (xy 95.25 52.07)
+		)
+		(stroke
+			(width 0)
+			(type default)
+		)
+	)
+	(wire
+		(pts
 			(xy 261.62 87.63) (xy 269.24 87.63)
 		)
@@
 		)
 		(stroke
+			(width 0)
+			(type default)
+		)
+	)
+	(wire
+		(pts
+			(xy 95.25 54.61) (xy 93.98 54.61)
+		)
+		(stroke

Commit message: Updates
Parts:
- removed NT1, NT2, NT3, NT4: NetTie_2, symbol Device:NetTie_2
Connections:
- net GND_CVSS is gone; now on net GND: C2.1, C5.1, C6.1, C8.1, U1.46
- net GND_DVSS is gone; now on net GND: C7.1, U1.50
- net GND_REFHM is gone; now on net GND: C3.1, U1.36

Commit message: Finished board
Parts:
- renumbered C1 to C201, C2 to C202, C3 to C203, C4 to C204, C5 to C205, C6 to C206, C7 to C207, C8 to C208, R1 to R201, U1 to U201
Changed lines of the file:
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@@
 	(label "Cell 14S PIN"
 		(at 77.47 49.53 0)
+		(fields_autoplaced yes)
 		(effects
 			(font
@@
 		(dnp no)
 		(fields_autoplaced yes)
-		(property "Reference" "C5"
+		(property "Reference" "C205"
 			(at 234.95 87.6299 90)
 			(effects
@@
 			(project "Project63_BMS_DaughterBoard"
 				(path "/325b096d-8e4c-4cdc-b4c5-634ea5e73c60/8ffa0956-e90f-44b3-af43-d8470a47be31"
-					(reference "C5")
+					(reference "C205")
 					(unit 1)
 				)
@@
 		(dnp no)
 		(fields_autoplaced yes)
-		(property "Reference" "C2"
+		(property "Reference" "C202"
 			(at 219.71 105.4099 90)
 			(effects
@@
 			(project "Project63_BMS_DaughterBoard"
 				(path "/325b096d-8e4c-4cdc-b4c5-634ea5e73c60/8ffa0956-e90f-44b3-af43-d8470a47be31"
-					(reference "C2")
+					(reference "C202")
 					(unit 1)
 				)
@@
 		(dnp no)
 		(fields_autoplaced yes)
-		(property "Reference" "U1"
+		(property "Reference" "U201"
 			(at 115.57 39.37 0)
 			(effects
@@
 			(project "Project63_BMS_DaughterBoard"
 				(path "/325b096d-8e4c-4cdc-b4c5-634ea5e73c60/8ffa0956-e90f-44b3-af43-d8470a47be31"
-					(reference "U1")
+					(reference "U201")
 					(unit 1)
 				)
@@
 		(dnp no)
 		(fields_autoplaced yes)
-		(property "Reference" "#PWR017"
+		(property "Reference" "#PWR0205"
 			(at 153.67 80.01 0)
 			(effects
@@
 			(project "Project63_BMS_DaughterBoard"
 				(path "/325b096d-8e4c-4cdc-b4c5-634ea5e73c60/8ffa0956-e90f-44b3-af43-d8470a47be31"
-					(reference "#PWR017")
+					(reference "#PWR0205")
 					(unit 1)
 				)
@@
 		(dnp no)
 		(fields_autoplaced yes)
-		(property "Reference" "#PWR016"
+		(property "Reference" "#PWR0203"
 			(at 142.24 144.78 0)
 			(effects
@@
 			(project "Project63_BMS_DaughterBoard"
 				(path "/325b096d-8e4c-4cdc-b4c5-634ea5e73c60/8ffa0956-e90f-44b3-af43-d8470a47be31"
-					(reference "#PWR016")
+					(reference "#PWR0203")
 					(unit 1)
 				)
@@
 		(dnp no)
 		(fields_autoplaced yes)
-		(property "Reference" "#PWR014"
+		(property "Reference" "#PWR0206"
 			(at 157.48 55.88 0)
 			(effects
@@
 			(project ""
 				(path "/325b096d-8e4c-4cdc-b4c5-634ea5e73c60/8ffa0956-e90f-44b3-af43-d8470a47be31"
-					(reference "#PWR014")
+					(reference "#PWR0206")
 					(unit 1)
 				)
@@
 		(dnp no)
 		(fields_autoplaced yes)
-		(property "Reference" "#PWR015"
+		(property "Reference" "#PWR0201"
 			(at 68.58 76.2 0)
 			(effects
@@
 			(project ""
 				(path "/325b096d-8e4c-4cdc-b4c5-634ea5e73c60/8ffa0956-e90f-44b3-af43-d8470a47be31"
-					(reference "#PWR015")
+					(reference "#PWR0201")
 					(unit 1)
 				)
@@
 		(dnp no)
 		(fields_autoplaced yes)
-		(property "Reference" "C4"
+		(property "Reference" "C204"
 			(at 227.33 120.6499 90)
 			(effects
@@
 			(project "Project63_BMS_DaughterBoard"
 				(path "/325b096d-8e4c-4cdc-b4c5-634ea5e73c60/8ffa0956-e90f-44b3-af43-d8470a47be31"
-					(reference "C4")
+					(reference "C204")
 					(unit 1)
 				)
@@
 		(dnp no)
 		(fields_autoplaced yes)
-		(property "Reference" "#PWR018"
+		(property "Reference" "#PWR0204"
 			(at 149.86 144.78 0)
 			(effects
@@
 			(project "Project63_BMS_DaughterBoard"
 				(path "/325b096d-8e4c-4cdc-b4c5-634ea5e73c60/8ffa0956-e90f-44b3-af43-d8470a47be31"
-					(reference "#PWR018")
+					(reference "#PWR0204")
 					(unit 1)
 				)
@@
 		(dnp no)
 		(fields_autoplaced yes)
-		(property "Reference" "C1"
+		(property "Reference" "C201"
 			(at 72.39 57.1499 90)
 			(effects
@@
 			(project "Project63_BMS_DaughterBoard"
 				(path "/325b096d-8e4c-4cdc-b4c5-634ea5e73c60/8ffa0956-e90f-44b3-af43-d8470a47be31"
-					(reference "C1")
+					(reference "C201")
 					(unit 1)
 				)
@@
 		(dnp no)
 		(fields_autoplaced yes)
-		(property "Reference" "R1"
+		(property "Reference" "R201"
 			(at 57.15 43.18 0)
 			(effects
@@
 			(project "Project63_BMS_DaughterBoard"
 				(path "/325b096d-8e4c-4cdc-b4c5-634ea5e73c60/8ffa0956-e90f-44b3-af43-d8470a47be31"
-					(reference "R1")
+					(reference "R201")
 					(unit 1)
 				)
@@
 		(dnp no)
 		(fields_autoplaced yes)
-		(property "Reference" "C8"
+		(property "Reference" "C208"
 			(at 267.97 102.8699 90)
 			(effects
@@
 			(project "Project63_BMS_DaughterBoard"
 				(path "/325b096d-8e4c-4cdc-b4c5-634ea5e73c60/8ffa0956-e90f-44b3-af43-d8470a47be31"
-					(reference "C8")
+					(reference "C208")
 					(unit 1)
 				)
@@
 		(dnp no)
 		(fields_autoplaced yes)
-		(property "Reference" "C7"
+		(property "Reference" "C207"
 			(at 265.43 82.5499 90)
 			(effects
@@
 			(project "Project63_BMS_DaughterBoard"
 				(path "/325b096d-8e4c-4cdc-b4c5-634ea5e73c60/8ffa0956-e90f-44b3-af43-d8470a47be31"
-					(reference "C7")
+					(reference "C207")
 					(unit 1)
 				)
@@
 		(dnp no)
 		(fields_autoplaced yes)
-		(property "Reference" "C3"
+		(property "Reference" "C203"
 			(at 222.25 142.2399 90)
 			(effects
@@
 			(project "Project63_BMS_DaughterBoard"
 				(path "/325b096d-8e4c-4cdc-b4c5-634ea5e73c60/8ffa0956-e90f-44b3-af43-d8470a47be31"
-					(reference "C3")
+					(reference "C203")
 					(unit 1)
 				)
@@
 		(dnp no)
 		(fields_autoplaced yes)
-		(property "Reference" "C6"
+		(property "Reference" "C206"
 			(at 252.73 138.4299 90)
 			(effects
@@
 			(project "Project63_BMS_DaughterBoard"
 				(path "/325b096d-8e4c-4cdc-b4c5-634ea5e73c60/8ffa0956-e90f-44b3-af43-d8470a47be31"
-					(reference "C6")
+					(reference "C206")
 					(unit 1)
 				)
@@
 		(dnp no)
 		(fields_autoplaced yes)
-		(property "Reference" "#PWR08"
+		(property "Reference" "#PWR0202"
 			(at 137.16 143.51 0)
 			(effects
@@
 			(project ""
 				(path "/325b096d-8e4c-4cdc-b4c5-634ea5e73c60/8ffa0956-e90f-44b3-af43-d8470a47be31"
-					(reference "#PWR08")
+					(reference "#PWR0202")
 					(unit 1)
 				)
