File: DaughterBoard/Test Points.kicad_sch (KiCad schematic)
At the start: 0 parts

Commit message: modhy commit
Parts:
- added TP1, TP10, TP11, TP12, TP13, TP14, TP15, TP16, TP17, TP2, TP3, TP4, TP5, TP6, TP7, TP8, TP9: ~, TestPoint:TestPoint_Keystone_5010-5014_Multipurpose, symbol Connector:TestPoint
Connections:
- new net AVDD: TP6.1
- new net BAT: TP8.1
- new net BBN: TP12.1
- new net BBP: TP11.1
- new net CVDD: TP5.1
- new net DVDD: TP10.1
- new net GND: TP1.1, TP2.1, TP3.1
- new net LDOIN: TP15.1
- new net NEG5V: TP16.1
- new net NFAULT: TP13.1
- new net NPNB: TP17.1
- new net REFHP: TP7.1
- new net RX: TP4.1
- new net TSREF: TP14.1
- new net TX: TP9.1

Commit message: 90% DOBO is done
Parts:
- removed TP1, TP10, TP11, TP12, TP13, TP14, TP15, TP16, TP17, TP2, TP3, TP4, TP5, TP6, TP7, TP8, TP9: ~, TestPoint:TestPoint_Keystone_5010-5014_Multipurpose, symbol Connector:TestPoint
- added TP1, TP10, TP11, TP12, TP13, TP14, TP2, TP3, TP4, TP5, TP6, TP7, TP8, TP9: 5012, TP5012:TP_5012, symbol 5012:5012
Connections:
- net AVDD: now also TP7.TP
- net BAT: now also TP5.TP
- net BBN: now also TP13.TP
- net BBP: now also TP12.TP
- net CVDD: now also TP9.TP
- net DVDD: now also TP11.TP
- net LDOIN: now also TP2.TP
- net NEG5V: now also TP3.TP
- net NFAULT: now also TP14.TP
- net NPNB: now also TP4.TP
- net REFHP: now also TP6.TP
- net RX: now also TP8.TP
- net TSREF: now also TP1.TP
- net TX: now also TP10.TP

Commit message: NPN is done
Changed lines of the file:
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@@
-	(wire
-		(pts
-			(xy 69.85 35.56) (xy 69.85 43.18)
-		)
-		(stroke
-			(width 0)
-			(type default)
-		)
-	)
 	(wire
 		(pts
@@
 	(wire
 		(pts
-			(xy 49.53 35.56) (xy 49.53 43.18)
-		)
-		(stroke
-			(width 0)
-			(type default)
-		)
-	)
-	(wire
-		(pts
 			(xy 217.17 102.87) (xy 231.14 102.87)
 		)
@@
 		(pts
 			(xy 93.98 52.07) (xy 107.95 52.07)
-		)
-		(stroke
-			(width 0)
-			(type default)
-		)
-	)
-	(wire
-		(pts
-			(xy 59.69 35.56) (xy 59.69 43.18)
 		)
 		(stroke
@@
 				(justify right)
 				(hide yes)
-			)
-		)
-	)
-	(symbol
-		(lib_id "power:GND")
-		(at 49.53 43.18 0)
-		(unit 1)
-		(exclude_from_sim no)
-		(in_bom yes)
-		(on_board yes)
-		(dnp no)
-		(fields_autoplaced yes)
-		(property "Reference" "#PWR01"
-			(at 49.53 49.53 0)
-			(effects
-				(font
-					(size 1.27 1.27)
-				)
-				(hide yes)
-			)
-		)
-		(property "Value" "GND"
-			(at 49.53 48.26 0)
-			(effects
-				(font
-					(size 1.27 1.27)
-				)
-			)
-		)
-		(property "Footprint" ""
-			(at 49.53 43.18 0)
-			(effects
-				(font
-					(size 1.27 1.27)
-				)
-				(hide yes)
-			)
-		)
-		(property "Datasheet" ""
-			(at 49.53 43.18 0)
-			(effects
-				(font
-					(size 1.27 1.27)
-				)
-				(hide yes)
-			)
-		)
-		(property "Description" "Power symbol creates a global label with name \"GND\" , ground"
-			(at 49.53 43.18 0)
-			(effects
-				(font
-					(size 1.27 1.27)
-				)
-				(hide yes)
-			)
-		)
-		(pin "1"
-		)
-		(instances
-			(project "Project63_BMS_DaughterBoard"
-				(path "/325b096d-8e4c-4cdc-b4c5-634ea5e73c60/f572dc6c-083b-4ebc-8b73-cb14171a47f1"
-					(reference "#PWR01")
-					(unit 1)
-				)
-			)
-		)
-	)
-	(symbol
-		(lib_id "power:GND")
-		(at 69.85 43.18 0)
-		(unit 1)
-		(exclude_from_sim no)
-		(in_bom yes)
-		(on_board yes)
-		(dnp no)
-		(fields_autoplaced yes)
-		(property "Reference" "#PWR03"
-			(at 69.85 49.53 0)
-			(effects
-				(font
-					(size 1.27 1.27)
-				)
-				(hide yes)
-			)
-		)
-		(property "Value" "GND"
-			(at 69.85 48.26 0)
-			(effects
-				(font
-					(size 1.27 1.27)
-				)
-			)
-		)
-		(property "Footprint" ""
-			(at 69.85 43.18 0)
-			(effects
-				(font
-					(size 1.27 1.27)
-				)
-				(hide yes)
-			)
-		)
-		(property "Datasheet" ""
-			(at 69.85 43.18 0)
-			(effects
-				(font
-					(size 1.27 1.27)
-				)
-				(hide yes)
-			)
-		)
-		(property "Description" "Power symbol creates a global label with name \"GND\" , ground"
-			(at 69.85 43.18 0)
-			(effects
-				(font
-					(size 1.27 1.27)
-				)
-				(hide yes)
-			)
-		)
-		(pin "1"
-		)
-		(instances
-			(project "Project63_BMS_DaughterBoard"
-				(path "/325b096d-8e4c-4cdc-b4c5-634ea5e73c60/f572dc6c-083b-4ebc-8b73-cb14171a47f1"
-					(reference "#PWR03")
-					(unit 1)
-				)
 			)
 		)
@@
 					(unit 1)
 				)
-			)
-		)
-	)
-	(symbol
-		(lib_id "power:GND")
-		(at 59.69 43.18 0)
-		(unit 1)
-		(exclude_from_sim no)
-		(in_bom yes)
-		(on_board yes)
-		(dnp no)
-		(fields_autoplaced yes)
-		(property "Reference" "#PWR02"
-			(at 59.69 49.53 0)
-			(effects
-				(font
-					(size 1.27 1.27)
-				)
-				(hide yes)
-			)
-		)
-		(property "Value" "GND"
-			(at 59.69 48.26 0)
-			(effects
-				(font
-					(size 1.27 1.27)
-				)
-			)
-		)
-		(property "Footprint" ""
-			(at 59.69 43.18 0)
-			(effects
-				(font
-					(size 1.27 1.27)
-				)
-				(hide yes)
-			)
-		)
-		(property "Datasheet" ""
-			(at 59.69 43.18 0)
-			(effects
-				(font
-					(size 1.27 1.27)
-				)
-				(hide yes)
-			)
-		)
-		(property "Description" "Power symbol creates a global label with name \"GND\" , ground"
-			(at 59.69 43.18 0)
-			(effects
-				(font
-					(size 1.27 1.27)
-				)
-				(hide yes)
-			)
-		)
-		(pin "1"
-		)
-		(instances
-			(project "Project63_BMS_DaughterBoard"
-				(path "/325b096d-8e4c-4cdc-b4c5-634ea5e73c60/f572dc6c-083b-4ebc-8b73-cb14171a47f1"
-					(reference "#PWR02")
-					(unit 1)
-				)

Commit message: C:/Program Files/Git/
Parts:
- TP1, TP10, TP11, TP12, TP13, TP14, TP2, TP3, TP4, TP5, TP6, TP7, TP8, TP9: Manufacturer Part Number (none) -> 5012
Changed lines of the file:
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@@
+			)
+		)
+		(property "Manufacturer Part Number" "5012"
+			(at 191.77 80.01 0)
+			(effects
+				(font
+					(size 1.27 1.27)
+				)
+				(hide yes)
 			)
 		)
@@
 			)
 		)
+		(property "Manufacturer Part Number" "5012"
+			(at 107.95 29.21 0)
+			(effects
+				(font
+					(size 1.27 1.27)
+				)
+				(hide yes)
+			)
+		)
 		(pin "TP"
 		)
@@
 			)
 		)
+		(property "Manufacturer Part Number" "5012"
+			(at 231.14 80.01 0)
+			(effects
+				(font
+					(size 1.27 1.27)
+				)
+				(hide yes)
+			)
+		)
 		(pin "TP"
 		)
@@
 			)
 		)
+		(property "Manufacturer Part Number" "5012"
+			(at 147.32 132.08 0)
+			(effects
+				(font
+					(size 1.27 1.27)
+				)
+				(hide yes)
+			)
+		)
 		(pin "TP"
 		)
@@
 			)
 		)
+		(property "Manufacturer Part Number" "5012"
+			(at 62.23 132.08 0)
+			(effects
+				(font
+					(size 1.27 1.27)
+				)
+				(hide yes)
+			)
+		)
 		(pin "TP"
 		)
@@
 			)
 		)
+		(property "Manufacturer Part Number" "5012"
+			(at 189.23 132.08 0)
+			(effects
+				(font
+					(size 1.27 1.27)
+				)
+				(hide yes)
+			)
+		)
 		(pin "TP"
 		)
@@
 			)
 		)
+		(property "Manufacturer Part Number" "5012"
+			(at 228.6 132.08 0)
+			(effects
+				(font
+					(size 1.27 1.27)
+				)
+				(hide yes)
+			)
+		)
 		(pin "TP"
 		)
@@
 			)
 		)
+		(property "Manufacturer Part Number" "5012"
+			(at 149.86 29.21 0)
+			(effects
+				(font
+					(size 1.27 1.27)
+				)
+				(hide yes)
+			)
+		)
 		(pin "TP"
 		)
@@
 			)
 		)
+		(property "Manufacturer Part Number" "5012"
+			(at 107.95 80.01 0)
+			(effects
+				(font
+					(size 1.27 1.27)
+				)
+				(hide yes)
+			)
+		)
 		(pin "TP"
 		)
@@
 			)
 		)
+		(property "Manufacturer Part Number" "5012"
+			(at 191.77 29.21 0)
+			(effects
+				(font
+					(size 1.27 1.27)
+				)
+				(hide yes)
+			)
+		)
 		(pin "TP"
 		)
@@
 			)
 		)
+		(property "Manufacturer Part Number" "5012"
+			(at 64.77 80.01 0)
+			(effects
+				(font
+					(size 1.27 1.27)
+				)
+				(hide yes)
+			)
+		)
 		(pin "TP"
 		)
@@
 			)
 		)
+		(property "Manufacturer Part Number" "5012"
+			(at 105.41 132.08 0)
+			(effects
+				(font
+					(size 1.27 1.27)
+				)
+				(hide yes)
+			)
+		)
 		(pin "TP"
 		)
@@
 			)
 		)
+		(property "Manufacturer Part Number" "5012"
+			(at 231.14 29.21 0)
+			(effects
+				(font
+					(size 1.27 1.27)
+				)
+				(hide yes)
+			)
+		)
 		(pin "TP"
 		)
@@
 				(hide yes)
 			)
+		)
+		(property "Manufacturer Part Number" "5012"
+			(at 149.86 80.01 0)
+			(effects
+				(font
+					(size 1.27 1.27)
+				)
+				(hide yes)
+			)

Commit message: tracing left
Parts:
- TP1, TP10, TP11, TP12, TP13, TP14, TP2, TP3, TP4, TP5, TP6, TP7, TP8, TP9: footprint TP5012:TP_5012 -> 5012:TP_5012
Changed lines of the file:
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@@
 			)
 		)
-		(property "Footprint" "TP5012:TP_5012"
+		(property "Footprint" "5012:TP_5012"
 			(at 191.77 80.01 0)
 			(effects
@@
 			)
 		)
-		(property "Footprint" "TP5012:TP_5012"
+		(property "Footprint" "5012:TP_5012"
 			(at 107.95 29.21 0)
 			(effects
@@
 			)
 		)
-		(property "Footprint" "TP5012:TP_5012"
+		(property "Footprint" "5012:TP_5012"
 			(at 231.14 80.01 0)
 			(effects
@@
 			)
 		)
-		(property "Footprint" "TP5012:TP_5012"
+		(property "Footprint" "5012:TP_5012"
 			(at 147.32 132.08 0)
 			(effects
@@
 			)
 		)
-		(property "Footprint" "TP5012:TP_5012"
+		(property "Footprint" "5012:TP_5012"
 			(at 62.23 132.08 0)
 			(effects
@@
 			)
 		)
-		(property "Footprint" "TP5012:TP_5012"
+		(property "Footprint" "5012:TP_5012"
 			(at 189.23 132.08 0)
 			(effects
@@
 			)
 		)
-		(property "Footprint" "TP5012:TP_5012"
+		(property "Footprint" "5012:TP_5012"
 			(at 228.6 132.08 0)
 			(effects
@@
 			)
 		)
-		(property "Footprint" "TP5012:TP_5012"
+		(property "Footprint" "5012:TP_5012"
 			(at 149.86 29.21 0)
 			(effects
@@
 			)
 		)
-		(property "Footprint" "TP5012:TP_5012"
+		(property "Footprint" "5012:TP_5012"
 			(at 107.95 80.01 0)
 			(effects
@@
 			)
 		)
-		(property "Footprint" "TP5012:TP_5012"
+		(property "Footprint" "5012:TP_5012"
 			(at 191.77 29.21 0)
 			(effects
@@
 			)
 		)
-		(property "Footprint" "TP5012:TP_5012"
+		(property "Footprint" "5012:TP_5012"
 			(at 64.77 80.01 0)
 			(effects
@@
 			)
 		)
-		(property "Footprint" "TP5012:TP_5012"
+		(property "Footprint" "5012:TP_5012"
 			(at 105.41 132.08 0)
 			(effects
@@
 			)
 		)
-		(property "Footprint" "TP5012:TP_5012"
+		(property "Footprint" "5012:TP_5012"
 			(at 231.14 29.21 0)
 			(effects
@@
 			)
 		)
-		(property "Footprint" "TP5012:TP_5012"
+		(property "Footprint" "5012:TP_5012"
 			(at 149.86 80.01 0)
 			(effects

Commit message: test
Parts:
- removed TP10, TP12, TP13, TP8: 5012, 5012:TP_5012, symbol 5012:5012

Commit message: Finished board
Parts:
- renumbered TP11 to TP501, TP1 to TP502, TP9 to TP503, TP2 to TP504, TP7 to TP505, TP3 to TP506, TP6 to TP507, TP14 to TP508, TP4 to TP509, TP5 to TP510
Changed lines of the file:
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@@
 		(dnp no)
 		(fields_autoplaced yes)
-		(property "Reference" "TP6"
+		(property "Reference" "TP507"
 			(at 194.31 78.7399 90)
 			(effects
@@
 			(project "Project63_BMS_DaughterBoard"
 				(path "/325b096d-8e4c-4cdc-b4c5-634ea5e73c60/f572dc6c-083b-4ebc-8b73-cb14171a47f1"
-					(reference "TP6")
+					(reference "TP507")
 					(unit 1)
 				)
@@
 		(dnp no)
 		(fields_autoplaced yes)
-		(property "Reference" "TP1"
+		(property "Reference" "TP502"
 			(at 110.49 27.9399 90)
 			(effects
@@
 			(project "Project63_BMS_DaughterBoard"
 				(path "/325b096d-8e4c-4cdc-b4c5-634ea5e73c60/f572dc6c-083b-4ebc-8b73-cb14171a47f1"
-					(reference "TP1")
+					(reference "TP502")
 					(unit 1)
 				)
@@
 		(dnp no)
 		(fields_autoplaced yes)
-		(property "Reference" "TP5"
+		(property "Reference" "TP510"
 			(at 233.68 78.7399 90)
 			(effects
@@
 			(project "Project63_BMS_DaughterBoard"
 				(path "/325b096d-8e4c-4cdc-b4c5-634ea5e73c60/f572dc6c-083b-4ebc-8b73-cb14171a47f1"
-					(reference "TP5")
+					(reference "TP510")
 					(unit 1)
 				)
@@
 		(dnp no)
 		(fields_autoplaced yes)
-		(property "Reference" "TP14"
+		(property "Reference" "TP508"
 			(at 231.14 130.8099 90)
 			(effects
@@
 			(project "Project63_BMS_DaughterBoard"
 				(path "/325b096d-8e4c-4cdc-b4c5-634ea5e73c60/f572dc6c-083b-4ebc-8b73-cb14171a47f1"
-					(reference "TP14")
+					(reference "TP508")
 					(unit 1)
 				)
@@
 		(dnp no)
 		(fields_autoplaced yes)
-		(property "Reference" "TP2"
+		(property "Reference" "TP504"
 			(at 152.4 27.9399 90)
 			(effects
@@
 			(project "Project63_BMS_DaughterBoard"
 				(path "/325b096d-8e4c-4cdc-b4c5-634ea5e73c60/f572dc6c-083b-4ebc-8b73-cb14171a47f1"
-					(reference "TP2")
+					(reference "TP504")
 					(unit 1)
 				)
@@
 		(dnp no)
 		(fields_autoplaced yes)
-		(property "Reference" "TP9"
+		(property "Reference" "TP503"
 			(at 110.49 78.7399 90)
 			(effects
@@
 			(project "Project63_BMS_DaughterBoard"
 				(path "/325b096d-8e4c-4cdc-b4c5-634ea5e73c60/f572dc6c-083b-4ebc-8b73-cb14171a47f1"
-					(reference "TP9")
+					(reference "TP503")
 					(unit 1)
 				)
@@
 		(dnp no)
 		(fields_autoplaced yes)
-		(property "Reference" "TP3"
+		(property "Reference" "TP506"
 			(at 194.31 27.9399 90)
 			(effects
@@
 			(project "Project63_BMS_DaughterBoard"
 				(path "/325b096d-8e4c-4cdc-b4c5-634ea5e73c60/f572dc6c-083b-4ebc-8b73-cb14171a47f1"
-					(reference "TP3")
+					(reference "TP506")
 					(unit 1)
 				)
@@
 		(dnp no)
 		(fields_autoplaced yes)
-		(property "Reference" "TP11"
+		(property "Reference" "TP501"
 			(at 107.95 130.8099 90)
 			(effects
@@
 			(project "Project63_BMS_DaughterBoard"
 				(path "/325b096d-8e4c-4cdc-b4c5-634ea5e73c60/f572dc6c-083b-4ebc-8b73-cb14171a47f1"
-					(reference "TP11")
+					(reference "TP501")
 					(unit 1)
 				)
@@
 		(dnp no)
 		(fields_autoplaced yes)
-		(property "Reference" "TP4"
+		(property "Reference" "TP509"
 			(at 233.68 27.9399 90)
 			(effects
@@
 			(project "Project63_BMS_DaughterBoard"
 				(path "/325b096d-8e4c-4cdc-b4c5-634ea5e73c60/f572dc6c-083b-4ebc-8b73-cb14171a47f1"
-					(reference "TP4")
+					(reference "TP509")
 					(unit 1)
 				)
@@
 		(dnp no)
 		(fields_autoplaced yes)
-		(property "Reference" "TP7"
+		(property "Reference" "TP505"
 			(at 152.4 78.7399 90)
 			(effects
@@
 			(project "Project63_BMS_DaughterBoard"
 				(path "/325b096d-8e4c-4cdc-b4c5-634ea5e73c60/f572dc6c-083b-4ebc-8b73-cb14171a47f1"
-					(reference "TP7")
+					(reference "TP505")
 					(unit 1)
 				)
