File: DaughterBoard/COMML.kicad_sch (KiCad schematic)
At the start: 36 parts, among them J1 430450200, J5 430450200

Commit message: Updates
Connections:
- net GND_CVSS renamed GND
Changed lines of the file:
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@@
+	)
+	(symbol
+		(lib_id "power:GND")
+		(at 354.33 96.52 0)
+		(unit 1)
+		(exclude_from_sim no)
+		(in_bom yes)
+		(on_board yes)
+		(dnp no)
+		(fields_autoplaced yes)
+		(property "Reference" "#PWR05"
+			(at 354.33 102.87 0)
+			(effects
+				(font
+					(size 1.27 1.27)
+				)
+				(hide yes)
+			)
+		)
+		(property "Value" "GND"
+			(at 354.33 101.6 0)
+			(effects
+				(font
+					(size 1.27 1.27)
+				)
+			)
+		)
+		(property "Footprint" ""
+			(at 354.33 96.52 0)
+			(effects
+				(font
+					(size 1.27 1.27)
+				)
+				(hide yes)
+			)
+		)
+		(property "Datasheet" ""
+			(at 354.33 96.52 0)
+			(effects
+				(font
+					(size 1.27 1.27)
+				)
+				(hide yes)
+			)
+		)
+		(property "Description" "Power symbol creates a global label with name \"GND\" , ground"
+			(at 354.33 96.52 0)
+			(effects
+				(font
+					(size 1.27 1.27)
+				)
+				(hide yes)
+			)
+		)
+		(pin "1"
+		)
+		(instances
+			(project "Project63_BMS_DaughterBoard"
+				(path "/325b096d-8e4c-4cdc-b4c5-634ea5e73c60/8d4a348c-1e09-4dff-8656-797547bf484e"
+					(reference "#PWR05")
+					(unit 1)
+				)
+			)
+		)
 	)
 	(symbol
@@
 	)
 	(symbol
-		(lib_id "power:GND")
-		(at 354.33 96.52 0)
-		(unit 1)
-		(exclude_from_sim no)
-		(in_bom yes)
-		(on_board yes)
-		(dnp no)
-		(fields_autoplaced yes)
-		(property "Reference" "#PWR013"
-			(at 354.33 102.87 0)
-			(effects
-				(font
-					(size 1.27 1.27)
-				)
-				(hide yes)
-			)
-		)
-		(property "Value" "GND_CVSS"
-			(at 356.87 97.7899 0)
-			(effects
-				(font
-					(size 1.27 1.27)
-				)
-				(justify left)
-			)
-		)
-		(property "Footprint" ""
-			(at 354.33 96.52 0)
-			(effects
-				(font
-					(size 1.27 1.27)
-				)
-				(hide yes)
-			)
-		)
-		(property "Datasheet" ""
-			(at 354.33 96.52 0)
-			(effects
-				(font
-					(size 1.27 1.27)
-				)
-				(hide yes)
-			)
-		)
-		(property "Description" "Power symbol creates a global label with name \"GND\" , ground"
-			(at 354.33 96.52 0)
-			(effects
-				(font
-					(size 1.27 1.27)
-				)
-				(hide yes)
-			)
-		)
-		(pin "1"
-		)
-		(instances
-			(project "Project63_BMS_DaughterBoard"
-				(path "/325b096d-8e4c-4cdc-b4c5-634ea5e73c60/8d4a348c-1e09-4dff-8656-797547bf484e"
-					(reference "#PWR013")
-					(unit 1)
-				)
-			)
-		)
-	)
-	(symbol
 		(lib_id "CRCW08050000Z0EAHP:CRCW08050000Z0EAHP")
 		(at 345.44 149.86 0)
@@
 	)
 	(symbol
+		(lib_id "power:GND")
+		(at 66.04 96.52 0)
+		(unit 1)
+		(exclude_from_sim no)
+		(in_bom yes)
+		(on_board yes)
+		(dnp no)
+		(fields_autoplaced yes)
+		(property "Reference" "#PWR04"
+			(at 66.04 102.87 0)
+			(effects
+				(font
+					(size 1.27 1.27)
+				)
+				(hide yes)
+			)
+		)
+		(property "Value" "GND"
+			(at 66.04 101.6 0)
+			(effects
+				(font
+					(size 1.27 1.27)
+				)
+			)
+		)
+		(property "Footprint" ""
+			(at 66.04 96.52 0)
+			(effects
+				(font
+					(size 1.27 1.27)
+				)
+				(hide yes)
+			)
+		)
+		(property "Datasheet" ""
+			(at 66.04 96.52 0)
+			(effects
+				(font
+					(size 1.27 1.27)
+				)
+				(hide yes)
+			)
+		)
+		(property "Description" "Power symbol creates a global label with name \"GND\" , ground"
+			(at 66.04 96.52 0)
+			(effects
+				(font
+					(size 1.27 1.27)
+				)
+				(hide yes)
+			)
+		)
+		(pin "1"
+		)
+		(instances
+			(project "Project63_BMS_DaughterBoard"
+				(path "/325b096d-8e4c-4cdc-b4c5-634ea5e73c60/8d4a348c-1e09-4dff-8656-797547bf484e"
+					(reference "#PWR04")
+					(unit 1)
+				)
+			)
+		)
+	)
+	(symbol
 		(lib_name "CRCW08050000Z0EAHP_2")
 		(lib_id "CRCW08050000Z0EAHP:CRCW08050000Z0EAHP")
@@
 					(unit 1)
 				)
-			)
-		)
-	)
-	(symbol
-		(lib_id "power:GND")
-		(at 66.04 96.52 0)
-		(unit 1)
-		(exclude_from_sim no)
-		(in_bom yes)
-		(on_board yes)
-		(dnp no)
-		(property "Reference" "#PWR012"
-			(at 66.04 102.87 0)
-			(effects
-				(font
-					(size 1.27 1.27)
-				)
-				(hide yes)
-			)
-		)
-		(property "Value" "GND_CVSS"
-			(at 61.214 104.648 0)
-			(effects
-				(font
-					(size 1.27 1.27)
-				)
-				(justify left)
-			)
-		)
-		(property "Footprint" ""
-			(at 66.04 96.52 0)
-			(effects
-				(font
-					(size 1.27 1.27)
-				)
-				(hide yes)
-			)
-		)
-		(property "Datasheet" ""
-			(at 66.04 96.52 0)
-			(effects
-				(font
-					(size 1.27 1.27)
-				)
-				(hide yes)
-			)
-		)
-		(property "Description" "Power symbol creates a global label with name \"GND\" , ground"
-			(at 66.04 96.52 0)
-			(effects
-				(font
-					(size 1.27 1.27)
-				)
-				(hide yes)
-			)
-		)
-		(pin "1"
-		)
-		(instances
-			(project "Project63_BMS_DaughterBoard"
-				(path "/325b096d-8e4c-4cdc-b4c5-634ea5e73c60/8d4a348c-1e09-4dff-8656-797547bf484e"
-					(reference "#PWR012")
-					(unit 1)
-				)

Commit message: Finished board
Parts:
- removed D1, D2: 24V, SOT23_PESD1_NEX, symbol PESD1CAN,215:PESD1CAN_215
- added D701, D702: 24V, Package_TO_SOT_SMD:SOT-23, symbol PESD1CAN,215:PESD1CAN_215
- renumbered C44 to C701, C43 to C702, C41 to C703, C40 to C704, C45 to C705, C42 to C706, C46 to C707, C47 to C708, FL1 to FL701, FL2 to FL702, J1 to J701, J5 to J702, R43 to R701, R44 to R702, R37 to R703, R38 to R704, R47 to R705, R48 to R706, R34 to R707, R35 to R708, R45 to R709, R46 to R710, R36 to R711, R49 to R712, R54 to R713, R55 to R714, R52 to R715, R53 to R716, R41 to R717, R42 to R718, R40 to R719, R39 to R720, R50 to R721, R51 to R722
Connections:
- net GND: now also D701.3, D702.3
- net at R703.2, R708.2: now also D701.1
- net at R717.2, R719.2: now also D702.1
- net at R718.2, R720.2: now also D702.2
- net at R704.2, R707.2: now also D701.2

Commit message: Both boards complete
Parts:
- C701, C702, C707, C708: JLC PCB Part # (none) -> C107194; Manufacturer Part Number 1206J2K00222 -> CC1206KKX7RCBB222
- C703, C704, C705, C706: JLC PCB Part # (none) -> C107081; Manufacturer Part Number CL10B221JB8NNNC -> CC0603KRX7R9BB221
- D701, D702: JLC PCB Part # (none) -> C314266; Manufacturer Part Number PESD1CAN_215 -> PESD24VL2BTN
- FL701, FL702: JLC PCB Part # (none) -> C488250
- J701, J702: now not fitted
- R701, R702, R705, R706, R709, R710, R713, R714, R715, R716, R721, R722: JLC PCB Part # (none) -> C844811
- R703, R704, R719, R720: JLC PCB Part # (none) -> C95177
- R707, R708, R717, R718: JLC PCB Part # (none) -> C844178
- R711, R712: JLC PCB Part # (none) -> C2907002; Manufacturer Part Number ERJ-3EKF1001V -> FRC0603F1001TS
