File: MotherBoard/FSAE_BMS.kicad_pcb (KiCad board)
At the start: 2 copper layers, 124 parts, among them IC501 BQ79600PWRQ1, J201 Conn_ARM_SWD_TagConnect_TC2030, J202 DM3AT-SF-PEJM5_40_, J301 1376357-3, J303 430450200, U201 STM32F205RBTx, U401 LMR51430, U402 LMR51430, U601 PTCAN1462DRQ1, U602 PTCAN1462DRQ1, Y201 16 Mhz

Commit message: Fixed relative paths + 90% footprints done + organized PCB for layout + found JLC part #s for manufacturing
Parts:
- added C502: 100p, Capacitor_SMD:C_0402_1005Metric, F.Cu at (115.5, 109.8)
- added C503: 100p, Capacitor_SMD:C_0402_1005Metric, F.Cu at (115.5, 111.8)
- added C505: 220n, Capacitor_SMD:C_0402_1005Metric, F.Cu at (115.5, 113.8)
- added C506: 2200p, Capacitor_SMD:C_0402_1005Metric, F.Cu at (115.5, 115.7)
- added C507: 2200p, Capacitor_SMD:C_0402_1005Metric, F.Cu at (115.5, 117.7)
- added C603: 4.7n, Capacitor_SMD:C_0402_1005Metric, F.Cu at (105.2, 137.0)
- added C607: 20pf, Capacitor_SMD:C_0402_1005Metric, F.Cu at (105.2, 139.0)
- added C608: 20pf, Capacitor_SMD:C_0402_1005Metric, F.Cu at (105.2, 140.9)
- added C609: 20pf, Capacitor_SMD:C_0402_1005Metric, F.Cu at (105.2, 142.9)
- added C610: 20pf, Capacitor_SMD:C_0402_1005Metric, F.Cu at (105.2, 144.9)
- added D401: GREEN, LED_SMD:LED_0603_1608Metric, F.Cu at (93.0, 76.9)
- added D402: GREEN, LED_SMD:LED_0603_1608Metric, F.Cu at (93.0, 79.5)
- added D403: D_Schottky, Diode_SMD:D_SMA, F.Cu at (62.2, 86.0)
- added D404: D_Schottky, Diode_SMD:D_SMA, F.Cu at (62.2, 90.6)
- added D409: RED, LED_SMD:LED_0603_1608Metric, F.Cu at (54.0, 72.3)
- added D501: RED, LED_SMD:LED_0603_1608Metric, F.Cu at (97.3, 106.3)
- added D701: 40V, Diode_SMD:D_SOD-123, F.Cu at (174.4, 132.2)
- added D702: 40V, Diode_SMD:D_SOD-123, F.Cu at (174.4, 135.6)
- added D703: 40V, Diode_SMD:D_SOD-123, F.Cu at (174.4, 138.9)
- added D704: 40V, Diode_SMD:D_SOD-123, F.Cu at (174.4, 142.3)
- added F401: 3A, Fuse:Fuse_1206_3216Metric, F.Cu at (69.1, 85.4)
- added F402: 3A, Fuse:Fuse_1206_3216Metric, F.Cu at (69.1, 88.7)
- added H101: MountingHole, MountingHole:MountingHole_3.2mm_M3, F.Cu at (25.0, 150.0)
- added H102: MountingHole, MountingHole:MountingHole_3.2mm_M3, F.Cu at (225.0, 20.0)
- added H103: MountingHole, MountingHole:MountingHole_3.2mm_M3, F.Cu at (225.0, 150.0)
- added H104: MountingHole, MountingHole:MountingHole_3.2mm_M3, F.Cu at (25.4, 25.4)
- added J302: Conn_01x04_Pin, Connector_PinHeader_2.54mm:PinHeader_1x04_P2.54mm_Vertical, F.Cu at (213.0, 76.2)
- added L501: WE-SLM, WE-SLM:WE-SLM, F.Cu at (98.6, 115.3)
- added Q701: Q_NMOS_GDS, Package_TO_SOT_SMD:TO-263-2, F.Cu at (164.5, 102.3)
- added Q702: Q_NPN_BEC, Package_TO_SOT_SMD:SOT-23, F.Cu at (173.9, 98.5)
- added Q703: Q_NPN_BEC, Package_TO_SOT_SMD:SOT-23, F.Cu at (173.9, 103.2)
- added Q704: Q_NMOS_GDS, Package_TO_SOT_SMD:TO-263-2, F.Cu at (164.5, 114.7)
- added Q705: Q_NPN_BEC, Package_TO_SOT_SMD:SOT-23, F.Cu at (173.9, 107.8)
- added Q706: Q_NMOS_GDS, Package_TO_SOT_SMD:TO-263-2, F.Cu at (164.5, 127.0)
- added Q708: Q_NPN_BEC, Package_TO_SOT_SMD:SOT-23, F.Cu at (173.9, 112.4)
- added Q709: Q_NMOS_GDS, Package_TO_SOT_SMD:TO-263-2, F.Cu at (164.5, 139.3)
- added R301: 22R, Resistor_SMD:R_0402_1005Metric, F.Cu at (216.8, 74.9)
- added R302: 22R, Resistor_SMD:R_0402_1005Metric, F.Cu at (216.8, 76.9)
- added R501: 1k, Resistor_SMD:R_0402_1005Metric, F.Cu at (106.8, 109.8)
- added R504: 100k, Resistor_SMD:R_0402_1005Metric, F.Cu at (106.8, 111.8)
- added R505: 10k, Resistor_SMD:R_0402_1005Metric, F.Cu at (106.8, 113.8)
- added R506: 10k, Resistor_SMD:R_0402_1005Metric, F.Cu at (106.8, 115.8)
- added R507: 10k, Resistor_SMD:R_0402_1005Metric, F.Cu at (106.8, 117.8)
- added R510: 10k, Resistor_SMD:R_0402_1005Metric, F.Cu at (109.7, 109.8)
- added R511: 100k, Resistor_SMD:R_0402_1005Metric, F.Cu at (109.7, 111.8)
- added R512: 0R, Resistor_SMD:R_0402_1005Metric, F.Cu at (109.7, 113.8)
- added R513: 0R, Resistor_SMD:R_0402_1005Metric, F.Cu at (109.7, 115.8)
- added R514: 0R, Resistor_SMD:R_0402_1005Metric, F.Cu at (109.7, 117.8)
- added R515: 0R, Resistor_SMD:R_0402_1005Metric, F.Cu at (112.6, 109.8)
- added R516: 0R, Resistor_SMD:R_0402_1005Metric, F.Cu at (112.6, 111.8)
- added R517: 0R, Resistor_SMD:R_0402_1005Metric, F.Cu at (112.6, 113.8)
- added R603: 10k, Resistor_SMD:R_0402_1005Metric, F.Cu at (96.5, 137.0)
- added R606: 10k, Resistor_SMD:R_0402_1005Metric, F.Cu at (96.5, 139.0)
- added R607: 10k, Resistor_SMD:R_0402_1005Metric, F.Cu at (96.5, 141.0)
- added R608: 10k, Resistor_SMD:R_0402_1005Metric, F.Cu at (96.5, 143.0)
- added R609: 10k, Resistor_SMD:R_0402_1005Metric, F.Cu at (96.5, 145.0)
- added R610: 10k, Resistor_SMD:R_0402_1005Metric, F.Cu at (99.4, 137.0)
- added R615: 10k, Resistor_SMD:R_0402_1005Metric, F.Cu at (99.4, 139.0)
- added R616: 10k, Resistor_SMD:R_0402_1005Metric, F.Cu at (99.4, 141.0)
- added R617: 0R, Resistor_SMD:R_0402_1005Metric, F.Cu at (99.4, 143.0)
- added R618: 0R, Resistor_SMD:R_0402_1005Metric, F.Cu at (99.4, 145.0)
- added R619: 0R, Resistor_SMD:R_0402_1005Metric, F.Cu at (102.3, 137.0)
- added R620: 0R, Resistor_SMD:R_0402_1005Metric, F.Cu at (102.3, 139.0)
- added R621: 0R, Resistor_SMD:R_0402_1005Metric, F.Cu at (102.3, 141.0)
- added R622: 0R, Resistor_SMD:R_0402_1005Metric, F.Cu at (102.3, 143.0)
- added R701: 100k, Resistor_SMD:R_0402_1005Metric, F.Cu at (172.9, 115.6)
- added R702: 10k, Resistor_SMD:R_0402_1005Metric, F.Cu at (172.9, 117.6)
- added R703: 10k, Resistor_SMD:R_0402_1005Metric, F.Cu at (172.9, 119.6)
- added R704: 100k, Resistor_SMD:R_0402_1005Metric, F.Cu at (172.9, 121.6)
- added R705: 10k, Resistor_SMD:R_0402_1005Metric, F.Cu at (172.9, 123.6)
- added R706: 100k, Resistor_SMD:R_0402_1005Metric, F.Cu at (172.9, 125.6)
- added R707: 10k, Resistor_SMD:R_0402_1005Metric, F.Cu at (172.9, 127.6)
- added R708: 100k, Resistor_SMD:R_0402_1005Metric, F.Cu at (172.9, 129.6)
- L402, L403: footprint SW_Inductor:IND_IHLP-6767DZ_VIS -> Inductor_SMD:L_Changjiang_FNR6045S
- R601, R602, R604, R605: value 0 -> 0R
- moved C202 229.0 mm to (51.0, 37.6)
- moved C205 229.0 mm to (51.0, 39.6)
- moved C207 229.0 mm to (51.0, 41.6)
- moved C209 229.0 mm to (51.0, 43.5)
- moved C211 229.0 mm to (51.0, 45.5)
- moved C212 229.0 mm to (51.0, 47.5)
- moved C214 229.0 mm to (51.0, 49.4)
- moved L201 229.0 mm to (51.0, 51.4)
- moved C419 221.9 mm to (51.8, 64.0)
- moved C420 221.9 mm to (51.8, 66.0)
- moved C415 220.2 mm to (37.2, 72.0)
- moved C416 220.2 mm to (37.2, 92.5)
- moved C417 220.2 mm to (37.2, 113.0)
- moved C418 220.2 mm to (37.2, 133.6)
- moved C201 180.4 mm to (54.4, 24.3)
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