File: MotherBoard/FSAE_BMS.kicad_pcb (KiCad board)
At the start: 4 copper layers, 115 x 125 mm, 234 parts, among them IC501 BQ79600PWRQ1, J201 Conn_ARM_SWD_TagConnect_TC2030, J202 DM3AT-SF-PEJM5_40_, J301 Conn_01x04_Pin, J302 Conn_01x04_Pin, J303 1376357-3, J304 430450200, J305 430450200, J306 Conn_01x02_Pin, Q701 Q_NPN_BEC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

Commit message: Fixed power routing mistake + finished BOM + generated manufacturing files
Parts:
- added G***: LOGO, LOGO, F.Cu at (112.8, 34.2)
- D403, D404, D407, D408: footprint Diode_SMD:D_SOD-323 -> Diode_SMD:D_SOD-123
- moved G*** 23.1 mm to (112.0, 84.2), turned to 0 degrees
- moved D501 20.5 mm to (131.3, 77.2)
- moved R501 19.9 mm to (132.7, 77.5), turned to -90 degrees
- moved D408 0.83 mm to (135.2, 97.2)
- moved D407 0.80 mm to (189.8, 99.7)
Routing:
- net BQ_NFAULT: track 24.0 -> 54.5 mm, vias 0 -> 2
- net +3V3: track 350.2 -> 371.7 mm
- net +5V: track 293.7 -> 294.5 mm
- net GND: track 86.6 -> 86.9 mm, vias 993 -> 944
Other:
- board text added: "STACK FAULT"

Commit message: Daughterboard 100% Complete + Edited Motherboard BOM
Parts:
- added F701: Fuse, Fuse:Fuse_1812_4532Metric, F.Cu at (157.3, 121.6)
- added F702: Fuse, Fuse:Fuse_1812_4532Metric, F.Cu at (184.0, 131.6)
- added F703: Fuse, Fuse:Fuse_1812_4532Metric, F.Cu at (133.9, 122.8)
- added F704: Fuse, Fuse:Fuse_1812_4532Metric, F.Cu at (134.7, 131.8)
- moved D703 3.11 mm to (200.2, 131.7)
- moved C703 3.11 mm to (200.1, 134.2)
- moved Q706 3.11 mm to (192.0, 131.3)
- moved C702 3.00 mm to (157.6, 117.1)
- moved D702 3.00 mm to (157.6, 114.6)
- moved C704 0.50 mm to (128.8, 132.4)
- moved D704 0.50 mm to (131.4, 132.4)
Connections:
- C701 pad 1: CHARGE_EN_HV -> Net-(D701-K)
- C702 pad 1: DISCHARGE_EN_HV -> Net-(D702-K)
- C703 pad 1: CHARGE_SAFE_HV -> Net-(D703-K)
- C704 pad 1: FAN_EN_HV -> Net-(D704-K)
- D701 pad 1: CHARGE_EN_HV -> Net-(D701-K)
- D702 pad 1: DISCHARGE_EN_HV -> Net-(D702-K)
- D703 pad 1: CHARGE_SAFE_HV -> Net-(D703-K)
- D704 pad 1: FAN_EN_HV -> Net-(D704-K)
- Q704 pad 2: CHARGE_EN_HV -> Net-(D701-K)
- Q705 pad 2: DISCHARGE_EN_HV -> Net-(D702-K)
- Q706 pad 2: CHARGE_SAFE_HV -> Net-(D703-K)
- Q708 pad 2: FAN_EN_HV -> Net-(D704-K)
Routing:
- net CHARGE_PWR_LV_ISO: track 290.9 -> 257.4 mm, vias 2 -> 4
- net READY_PWR_LV_ISO: track 262.5 -> 230.5 mm, vias 2 -> 4
- net CHARGE_EN_HV: track 29.6 -> 22.1 mm
- net CHARGE_SAFE_HV: track 32.5 -> 25.7 mm
- net Net-(D703-K): track 0.00 -> 5.84 mm
- net Net-(D702-K): track 0.00 -> 5.17 mm
- net FAN_EN_HV: track 21.7 -> 16.6 mm
- net DISCHARGE_EN_HV: track 8.74 -> 3.66 mm
- net Net-(D704-K): track 0.00 -> 4.62 mm
- net Net-(D701-K): track 0.00 -> 3.90 mm
- net Net-(Q703-C): track 5.91 -> 8.60 mm
- net ISO_CAN1+: track 45.9 -> 45.1 mm
- net +3V3: track 371.7 -> 371.1 mm
- net ISO_CAN1-: track 46.4 -> 45.9 mm
- net GND: vias 944 -> 925
- added copper zone on F.Cu, net Net-(D701-K)
- added copper zone on F.Cu, net Net-(D702-K)
- added copper zone on F.Cu, net Net-(D703-K)
- added copper zone on F.Cu, net Net-(D704-K)
- removed copper zone on F.Cu, net CHARGE_EN_HV
- removed copper zone on F.Cu, net CHARGE_SAFE_HV
- removed copper zone on F.Cu, net DISCHARGE_EN_HV
- removed copper zone on F.Cu, net FAN_EN_HV
