File: MotherBoard/Relay Drivers.kicad_sch (KiCad schematic)
At the start: 24 parts, among them Q701 Q_NMOS_GDS, Q702 Q_NPN_BEC, Q703 Q_NPN_BEC, Q704 Q_NMOS_GDS, Q705 Q_NPN_BEC, Q706 Q_NMOS_GDS, Q708 Q_NPN_BEC, Q709 Q_NMOS_GDS

Commit message: Finished layout need to route
Parts:
- renumbered Q708 to Q701, Q709 to Q704, Q701 to Q705, Q704 to Q706, Q705 to Q707, Q706 to Q708, R702 to R701, R703 to R702, R705 to R703, R701 to R704, R704 to R705
Changed lines of the file:
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@@
 		(dnp no)
 		(fields_autoplaced yes)
-		(property "Reference" "#PWR0701"
+		(property "Reference" "#PWR0707"
 			(at 78.74 63.5 0)
 			(effects
@@
 			(project ""
 				(path "/335e81e9-b957-4266-8116-dde74329bfca/2f5b3e7e-a53c-4958-9d9b-49ffd0a960f5"
-					(reference "#PWR0701")
+					(reference "#PWR0707")
 					(unit 1)
 				)
@@
 		(dnp no)
 		(fields_autoplaced yes)
-		(property "Reference" "R705"
+		(property "Reference" "R703"
 			(at 53.34 146.05 90)
 			(effects
@@
 			(project "FSAE_BMS"
 				(path "/335e81e9-b957-4266-8116-dde74329bfca/2f5b3e7e-a53c-4958-9d9b-49ffd0a960f5"
-					(reference "R705")
+					(reference "R703")
 					(unit 1)
 				)
@@
 		(on_board yes)
 		(dnp no)
-		(property "Reference" "Q706"
+		(property "Reference" "Q708"
 			(at 196.85 43.1799 0)
 			(effects
@@
 			(project "FSAE_BMS"
 				(path "/335e81e9-b957-4266-8116-dde74329bfca/2f5b3e7e-a53c-4958-9d9b-49ffd0a960f5"
-					(reference "Q706")
+					(reference "Q708")
 					(unit 1)
 				)
@@
 		(dnp no)
 		(fields_autoplaced yes)
-		(property "Reference" "R701"
+		(property "Reference" "R704"
 			(at 68.58 38.0999 0)
 			(effects
@@
 			(project ""
 				(path "/335e81e9-b957-4266-8116-dde74329bfca/2f5b3e7e-a53c-4958-9d9b-49ffd0a960f5"
-					(reference "R701")
+					(reference "R704")
 					(unit 1)
 				)
@@
 		(dnp no)
 		(fields_autoplaced yes)
-		(property "Reference" "#PWR0707"
+		(property "Reference" "#PWR0705"
 			(at 66.04 139.7 0)
 			(effects
@@
 			(project "FSAE_BMS"
 				(path "/335e81e9-b957-4266-8116-dde74329bfca/2f5b3e7e-a53c-4958-9d9b-49ffd0a960f5"
-					(reference "#PWR0707")
+					(reference "#PWR0705")
 					(unit 1)
 				)
@@
 		(on_board yes)
 		(dnp no)
-		(property "Reference" "Q704"
+		(property "Reference" "Q706"
 			(at 82.55 144.7799 0)
 			(effects
@@
 			(project "FSAE_BMS"
 				(path "/335e81e9-b957-4266-8116-dde74329bfca/2f5b3e7e-a53c-4958-9d9b-49ffd0a960f5"
-					(reference "Q704")
+					(reference "Q706")
 					(unit 1)
 				)
@@
 		(on_board yes)
 		(dnp no)
-		(property "Reference" "Q708"
+		(property "Reference" "Q701"
 			(at 68.58 49.5299 0)
 			(effects
@@
 			(project ""
 				(path "/335e81e9-b957-4266-8116-dde74329bfca/2f5b3e7e-a53c-4958-9d9b-49ffd0a960f5"
-					(reference "Q708")
+					(reference "Q701")
 					(unit 1)
 				)
@@
 		(dnp no)
 		(fields_autoplaced yes)
-		(property "Reference" "R704"
+		(property "Reference" "R705"
 			(at 68.58 88.8999 0)
 			(effects
@@
 			(project "FSAE_BMS"
 				(path "/335e81e9-b957-4266-8116-dde74329bfca/2f5b3e7e-a53c-4958-9d9b-49ffd0a960f5"
-					(reference "R704")
+					(reference "R705")
 					(unit 1)
 				)
@@
 		(dnp no)
 		(fields_autoplaced yes)
-		(property "Reference" "#PWR0705"
+		(property "Reference" "#PWR0704"
 			(at 66.04 114.3 0)
 			(effects
@@
 			(project "FSAE_BMS"
 				(path "/335e81e9-b957-4266-8116-dde74329bfca/2f5b3e7e-a53c-4958-9d9b-49ffd0a960f5"
-					(reference "#PWR0705")
+					(reference "#PWR0704")
 					(unit 1)
 				)
@@
 		(dnp no)
 		(fields_autoplaced yes)
-		(property "Reference" "R702"
+		(property "Reference" "R701"
 			(at 53.34 44.45 90)
 			(effects
@@
 			(project "FSAE_BMS"
 				(path "/335e81e9-b957-4266-8116-dde74329bfca/2f5b3e7e-a53c-4958-9d9b-49ffd0a960f5"
-					(reference "R702")
+					(reference "R701")
 					(unit 1)
 				)
@@
 		(dnp no)
 		(fields_autoplaced yes)
-		(property "Reference" "R703"
+		(property "Reference" "R702"
 			(at 53.34 95.25 90)
 			(effects
@@
 			(project "FSAE_BMS"
 				(path "/335e81e9-b957-4266-8116-dde74329bfca/2f5b3e7e-a53c-4958-9d9b-49ffd0a960f5"
-					(reference "R703")
+					(reference "R702")
 					(unit 1)
 				)
@@
 		(on_board yes)
 		(dnp no)
-		(property "Reference" "Q709"
+		(property "Reference" "Q704"
 			(at 82.55 43.1799 0)
 			(effects
@@
 			(project ""
 				(path "/335e81e9-b957-4266-8116-dde74329bfca/2f5b3e7e-a53c-4958-9d9b-49ffd0a960f5"
-					(reference "Q709")
+					(reference "Q704")
 					(unit 1)
 				)
@@
 		(on_board yes)
 		(dnp no)
-		(property "Reference" "Q705"
+		(property "Reference" "Q707"
 			(at 182.88 49.5299 0)
 			(effects
@@
 			(project "FSAE_BMS"
 				(path "/335e81e9-b957-4266-8116-dde74329bfca/2f5b3e7e-a53c-4958-9d9b-49ffd0a960f5"
-					(reference "Q705")
+					(reference "Q707")
 					(unit 1)
 				)
@@
 		(dnp no)
 		(fields_autoplaced yes)
-		(property "Reference" "#PWR0704"
+		(property "Reference" "#PWR0703"
 			(at 66.04 88.9 0)
 			(effects
@@
 			(project "FSAE_BMS"
 				(path "/335e81e9-b957-4266-8116-dde74329bfca/2f5b3e7e-a53c-4958-9d9b-49ffd0a960f5"
-					(reference "#PWR0704")
+					(reference "#PWR0703")
 					(unit 1)
 				)
@@
 		(on_board yes)
 		(dnp no)
-		(property "Reference" "Q701"
+		(property "Reference" "Q705"
 			(at 82.55 93.9799 0)
 			(effects
@@
 			(project "FSAE_BMS"
 				(path "/335e81e9-b957-4266-8116-dde74329bfca/2f5b3e7e-a53c-4958-9d9b-49ffd0a960f5"
-					(reference "Q701")
+					(reference "Q705")
 					(unit 1)
 				)
@@
 		(dnp no)
 		(fields_autoplaced yes)
-		(property "Reference" "#PWR0703"
+		(property "Reference" "#PWR0701"
 			(at 66.04 38.1 0)
 			(effects
@@
 			(project ""
 				(path "/335e81e9-b957-4266-8116-dde74329bfca/2f5b3e7e-a53c-4958-9d9b-49ffd0a960f5"
-					(reference "#PWR0703")
+					(reference "#PWR0701")
 					(unit 1)
 				)
@@
 		(dnp no)
 		(fields_autoplaced yes)
-		(property "Reference" "#PWR0708"
+		(property "Reference" "#PWR0706"
 			(at 66.04 165.1 0)
 			(effects
@@
 			(project "FSAE_BMS"
 				(path "/335e81e9-b957-4266-8116-dde74329bfca/2f5b3e7e-a53c-4958-9d9b-49ffd0a960f5"
-					(reference "#PWR0708")
+					(reference "#PWR0706")
 					(unit 1)
 				)
@@
 		(dnp no)
 		(fields_autoplaced yes)
-		(property "Reference" "#PWR0706"
+		(property "Reference" "#PWR0708"
 			(at 78.74 114.3 0)
 			(effects
@@
 			(project "FSAE_BMS"
 				(path "/335e81e9-b957-4266-8116-dde74329bfca/2f5b3e7e-a53c-4958-9d9b-49ffd0a960f5"
-					(reference "#PWR0706")
-					(unit 1)
-				)
+					(reference "#PWR0708")
+					(unit 1)
+				)

Commit message: Finished motherboard. Need to review BOM
Parts:
- added R701, R702, R703, R710: 10k, Resistor_SMD:R_0402_1005Metric, symbol Device:R_US
- renumbered R701 to R704, R702 to R705, R703 to R706, R704 to R707, R705 to R708, R706 to R709, R707 to R711, R708 to R712
Connections:
- net CHARGE_EN_LV: now also R701.2
- net CHARGE_SAFE_LV: now also R703.2
- net DISCHARGE_EN_LV: now also R702.2
- net FAN_EN_LV: now also R710.2
- net GND: now also R701.1, R702.1, R703.1, R710.1
- net +12V renamed VBUS
