File: MotherBoard/BQ79600.kicad_sch (KiCad schematic)
At the start: 48 parts, among them IC501 BQ79600PWRQ1

Commit message: Finished motherboard. Need to review BOM
Parts:
- C508: footprint Capacitor_SMD:C_0603_1608Metric -> Capacitor_SMD:C_0402_1005Metric; Manufacturer_Part_Number CL10B224KA8NNNC -> CL05A224KA5NNNC
- R520, R521, R522, R523: now not fitted
Connections:
- net COMLN: now also C505.2, R504.1, R512.1; no longer C506.1, R505.2, R513.1
- net COMLP: now also C506.1, R505.2, R513.1; no longer C505.2, R504.1, R512.1
- net ISO_COMLN: now also R526.2; no longer R527.2
- net ISO_COMLP: now also R527.2; no longer R526.2

Commit message: Fixed power routing mistake + finished BOM + generated manufacturing files
Parts:
- D502, D503, D504, D505: JLC (none) -> C668923; Manufacturer_Part_Number (none) -> ESD5V0D3B-TP

Commit message: Both boards complete
Parts:
- C501, C502: JLCPCB Part # (none) -> C60133
- C503, C504, C505, C506: JLCPCB Part # (none) -> C1546
- C507, C513: JLCPCB Part # (none) -> C21120
- C508: JLCPCB Part # (none) -> C47129
- C509, C510, C511, C512: JLCPCB Part # (none) -> C28260
- D501: JLCPCB Part # (none) -> C2286
- D502, D503, D504, D505: JLC C668923 -> (none); JLCPCB Part # (none) -> C668923
- IC501: JLCPCB Part # (none) -> C2869947
- L501, L502: JLCPCB Part # (none) -> C488250
- R501: JLCPCB Part # (none) -> C11702
- R502, R503, R504, R505: JLCPCB Part # (none) -> C23065
- R506, R515: JLCPCB Part # (none) -> C25741
- R507, R508, R509, R514: JLCPCB Part # (none) -> C2930027; Manufacturer_Part_Number 0402WGF1001TCE -> FRC0603J103TS
- R510, R511, R512, R513: JLCPCB Part # (none) -> C18019; Manufacturer_Part_Number C18019 -> 1206W4F510JT5E
- R516, R517, R518, R519, R524, R525, R526, R527: JLCPCB Part # (none) -> C17477
Changed lines of the file:
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@@
 			)
 		)
-		(property "JLC" ""
+		(property "JLCPCB Part #" "C60133"
 			(at 53.34 114.3 0)
 			(effects
@@
 			)
 		)
-		(property "JLC" ""
+		(property "JLCPCB Part #" "C21120"
 			(at 95.25 72.39 0)
 			(effects
@@
 			)
 		)
-		(property "JLC" ""
+		(property "JLCPCB Part #" "C488250"
 			(at 123.19 114.3 0)
 			(effects
@@
 			)
 		)
-		(property "Manufacturer_Part_Number" "0402WGF1001TCE"
+		(property "Manufacturer_Part_Number" "FRC0603J103TS"
 			(at 67.31 39.37 0)
 			(effects
@@
 			)
 		)
-		(property "JLC" ""
+		(property "JLCPCB Part #" "C2930027"
 			(at 67.31 39.37 0)
 			(effects
@@
 			)
 		)
-		(property "JLC" ""
+		(property "JLCPCB Part #" "C17477"
 			(at 139.7 143.51 0)
 			(effects
@@
 			)
 		)
-		(property "JLC" ""
+		(property "JLCPCB Part #" "C17477"
 			(at 139.7 104.14 0)
 			(effects
@@
 			)
 		)
-		(property "JLC" "C668923"
+		(property "Manufacturer_Part_Number" "ESD5V0D3B-TP"
 			(at 85.09 148.59 0)
 			(effects
@@
 			)
 		)
-		(property "Manufacturer_Part_Number" "ESD5V0D3B-TP"
+		(property "JLCPCB Part #" "C668923"
 			(at 85.09 148.59 0)
 			(effects
@@
 			)
 		)
-		(property "JLC" ""
+		(property "JLCPCB Part #" "C28260"
 			(at 106.68 143.51 0)
 			(effects
@@
 			)
 		)
-		(property "JLC" "C668923"
+		(property "Manufacturer_Part_Number" "ESD5V0D3B-TP"
 			(at 85.09 158.75 0)
 			(effects
@@
 			)
 		)
-		(property "Manufacturer_Part_Number" "ESD5V0D3B-TP"
+		(property "JLCPCB Part #" "C668923"
 			(at 85.09 158.75 0)
 			(effects
@@
 			)
 		)
-		(property "Manufacturer_Part_Number" "C18019"
+		(property "Manufacturer_Part_Number" "1206W4F510JT5E"
 			(at 73.66 163.83 0)
 			(effects
@@
 			)
 		)
-		(property "JLC" ""
+		(property "JLCPCB Part #" "C18019"
 			(at 73.66 163.83 0)
 			(effects
@@
 			)
 		)
-		(property "JLC" ""
+		(property "JLCPCB Part #" "C23065"
 			(at 45.72 109.22 0)
 			(effects
@@
 			)
 		)
-		(property "JLC" ""
+		(property "JLCPCB Part #" "C17477"
 			(at 96.52 104.14 0)
 			(effects
@@
 			)
 		)
-		(property "JLC" ""
+		(property "JLCPCB Part #" "C23065"
 			(at 45.72 158.75 0)
 			(effects
@@
 			)
 		)
-		(property "Manufacturer_Part_Number" "C18019"
+		(property "Manufacturer_Part_Number" "1206W4F510JT5E"
 			(at 73.66 143.51 0)
 			(effects
@@
 			)
 		)
-		(property "JLC" ""
+		(property "JLCPCB Part #" "C18019"
 			(at 73.66 143.51 0)
 			(effects
@@
 			)
 		)
-		(property "JLC" ""
+		(property "JLCPCB Part #" "C11702"
 			(at 40.64 34.29 0)
 			(effects
@@
 			)
 		)
-		(property "JLC" ""
+		(property "JLCPCB Part #" "C25741"
 			(at 85.09 39.37 0)
 			(effects
@@
 			)
 		)
-		(property "JLC" ""
+		(property "JLCPCB Part #" "C23065"
 			(at 45.72 119.38 0)
 			(effects
@@
 			)
 		)
-		(property "JLC" ""
-			(at 123.19 139.7 0)
-			(effects
-				(font
-					(size 1.27 1.27)
-				)
-				(hide yes)
-			)
-		)
 		(pin "2"
 		)
@@
 			)
 		)
-		(property "JLC" "C668923"
+		(property "Manufacturer_Part_Number" "ESD5V0D3B-TP"
 			(at 85.09 109.22 0)
 			(effects
@@
 			)
 		)
-		(property "Manufacturer_Part_Number" "ESD5V0D3B-TP"
+		(property "JLCPCB Part #" "C668923"
 			(at 85.09 109.22 0)
 			(effects
@@
 			)
 		)
-		(property "JLC" ""
+		(property "JLCPCB Part #" "C17477"
 			(at 96.52 143.51 0)
 			(effects
@@
 			)
 		)
-		(property "JLC" ""
+		(property "JLCPCB Part #" "C1546"
 			(at 60.96 109.22 0)
 			(effects
@@
 			)
 		)
-		(property "JLC" ""
+		(property "JLCPCB Part #" "C28260"
 			(at 106.68 104.14 0)
 			(effects
@@
 			)
 		)
-		(property "JLC" ""
+		(property "JLCPCB Part #" "C28260"
 			(at 106.68 163.83 0)
 			(effects
@@
 			)
 		)
-		(property "JLC" ""
+		(property "JLCPCB Part #" "C488250"
 			(at 123.19 153.67 0)
 			(effects
@@
 			)
 		)
-		(property "Manufacturer_Part_Number" "0402WGF1001TCE"
+		(property "Manufacturer_Part_Number" "FRC0603J103TS"
 			(at 58.42 39.37 0)
 			(effects
@@
 			)
 		)
-		(property "JLC" ""
+		(property "JLCPCB Part #" "C2930027"
 			(at 58.42 39.37 0)
 			(effects
@@
 			)
 		)
-		(property "JLC" ""
-			(at 123.19 100.33 0)
-			(effects
-				(font
-					(size 1.27 1.27)
-				)
-				(hide yes)
-			)
-		)
 		(pin "2"
 		)
@@
 			)
 		)
-		(property "Manufacturer_Part_Number" "0402WGF1001TCE"
+		(property "Manufacturer_Part_Number" "FRC0603J103TS"
 			(at 76.2 39.37 0)
 			(effects
@@
 			)
 		)
-		(property "JLC" ""
+		(property "JLCPCB Part #" "C2930027"
 			(at 76.2 39.37 0)
 			(effects
@@
 			)
 		)
-		(property "JLC" ""
+		(property "JLCPCB Part #" "C23065"
 			(at 45.72 148.59 0)
 			(effects
@@
 			)
 		)
-		(property "Manufacturer_Part_Number" "C18019"
+		(property "Manufacturer_Part_Number" "1206W4F510JT5E"
 			(at 73.66 124.46 0)
 			(effects
@@
 			)
 		)
-		(property "JLC" ""
+		(property "JLCPCB Part #" "C18019"
 			(at 73.66 124.46 0)
 			(effects
@@
 			)
 		)
-		(property "JLC" ""
+		(property "JLCPCB Part #" "C1546"
 			(at 60.96 158.75 0)
 			(effects
@@
 			)
 		)
-		(property "JLC" ""
+		(property "JLCPCB Part #" "C17477"
 			(at 96.52 124.46 0)
 			(effects
@@
 			)
 		)
-		(property "JLC" ""
+		(property "JLCPCB Part #" "C21120"
 			(at 158.75 59.69 0)
 			(effects
@@
 			)
 		)
-		(property "JLC" ""
+		(property "JLCPCB Part #" "C1546"
 			(at 60.96 148.59 0)
 			(effects
@@
 			)
 		)
-		(property "JLC" ""
+		(property "JLCPCB Part #" "C17477"
 			(at 139.7 163.83 0)
 			(effects
@@
 			)
 		)
-		(property "JLC" ""
+		(property "JLCPCB Part #" "C28260"
 			(at 106.68 124.46 0)
 			(effects
@@
 			)
 		)
-		(property "JLC" ""
-			(at 123.19 167.64 0)
-			(effects
-				(font
-					(size 1.27 1.27)
-				)
-				(hide yes)
-			)
-		)
 		(pin "2"
 		)
@@
 			)
 		)
-		(property "JLC" ""
+		(property "JLCPCB Part #" "C1546"
 			(at 60.96 119.38 0)
 			(effects
@@
 			)
 		)
-		(property "JLC" ""
+		(property "JLCPCB Part #" "C60133"
 			(at 53.34 153.67 0)
 			(effects
@@
 			)
 		)
-		(property "JLC" ""
+		(property "JLCPCB Part #" "C2286"
 			(at 40.64 43.18 0)
 			(effects
@@
 			)
 		)
-		(property "JLC" ""
+		(property "JLCPCB Part #" "C25741"
 			(at 49.53 39.37 0)
 			(effects
@@
 			)
 		)
-		(property "Manufacturer_Part_Number" "C18019"
+		(property "Manufacturer_Part_Number" "1206W4F510JT5E"
 			(at 73.66 104.14 0)
 			(effects
@@
 			)
 		)
-		(property "JLC" ""
+		(property "JLCPCB Part #" "C18019"
 			(at 73.66 104.14 0)
 			(effects
@@
 			)
 		)
-		(property "JLC" ""
+		(property "JLCPCB Part #" "C17477"
 			(at 139.7 124.46 0)
 			(effects
@@
 			)
 		)
-		(property "Manufacturer_Part_Number" "0402WGF1001TCE"
+		(property "Manufacturer_Part_Number" "FRC0603J103TS"
 			(at 72.39 72.39 0)
 			(effects
@@
 			)
 		)
-		(property "JLC" ""
+		(property "JLCPCB Part #" "C2930027"
 			(at 72.39 72.39 0)
 			(effects
@@
 			)
 		)
-		(property "JLC" ""
+		(property "JLCPCB Part #" "C2869947"
 			(at 96.52 46.99 0)
 			(effects
@@
 			)
 		)
-		(property "JLC" ""
+		(property "JLCPCB Part #" "C47129"
 			(at 99.06 35.56 0)
 			(effects
@@
 			)
 		)
-		(property "JLC" ""
-			(at 123.19 128.27 0)
-			(effects
-				(font
-					(size 1.27 1.27)
-				)
-				(hide yes)
-			)
-		)
 		(pin "2"
 		)
@@
 			)
 		)
-		(property "JLC" "C668923"
+		(property "Manufacturer_Part_Number" "ESD5V0D3B-TP"
 			(at 85.09 119.38 0)
 			(effects
@@
 			)
 		)
-		(property "Manufacturer_Part_Number" "ESD5V0D3B-TP"
+		(property "JLCPCB Part #" "C668923"
 			(at 85.09 119.38 0)
 			(effects
@@
 			)
 		)
-		(property "JLC" ""
+		(property "JLCPCB Part #" "C17477"
 			(at 96.52 163.83 0)
 			(effects
