File: MotherBoard/CAN_TRANCEIVER.kicad_sch (KiCad schematic)
At the start: 40 parts, among them U601 PTCAN1462DRQ1, U602 PTCAN1462DRQ1

Commit message: Layout 90% complete
Parts:
- R601, R602, R611, R612: footprint Resistor_SMD:R_2512_6332Metric -> Resistor_SMD:R_1210_3225Metric; Manufacturer_Part_Number 25121WF604JT4E -> AC1210FR-0760R4L
- R604, R605, R609, R610: footprint Resistor_SMD:R_0805_2012Metric -> Resistor_SMD:R_1206_3216Metric; Manufacturer_Part_Number 0805W8F0000T5E -> HP06W2J0000T5E
Connections:
- net CANL_1: now also R604.1; no longer R610.1
- net CANL_2: now also R610.1; no longer R604.1
- net ISO_CAN1+: now also R601.2; no longer R611.2
- net ISO_CAN1-: now also R602.1, R604.2; no longer R610.2, R612.1
- net ISO_CAN2+: now also R611.2; no longer R601.2
- net ISO_CAN2-: now also R610.2, R612.1; no longer R602.1, R604.2
- net at R601.1, R602.2: now also C603.1; no longer C606.1
- net at R611.1, R612.2: now also C606.1; no longer C603.1

Commit message: Finished layout need to route
Parts:
- renumbered C606 to C604, C604 to C605, C607 to C606, C608 to C607, C615 to C608, C616 to C609, C605 to C610, C613 to C612, C619 to C613, C609 to C614, C610 to C615, C612 to C616, C614 to C617, C620 to C618, C617 to C619, C618 to C620, R603 to R601, R606 to R602, R609 to R603, R610 to R606, R601 to R609, R602 to R610, R617 to R613, R618 to R614, R619 to R615, R620 to R616, R621 to R617, R622 to R618

Commit message: Both boards complete
Parts:
- C601, C602, C605, C610: JLCPCB Part # (none) -> C1554
- C603, C604: JLCPCB Part # (none) -> C281757
- C606, C607, C608, C609: value 20pf -> 20p; JLCPCB Part # (none) -> C1554
- C611, C612, C616, C617: JLCPCB Part # (none) -> C1525
- C613, C615, C618, C620: JLCPCB Part # (none) -> C29266
- C614, C619: JLCPCB Part # (none) -> C19702
- R601, R602, R607, R608: JLCPCB Part # (none) -> C2930027; Manufacturer_Part_Number 0402WGF1001TCE -> FRC0603J103TS
- R603, R604, R605, R606: JLCPCB Part # (none) -> C473612
- R609, R610, R611, R612: JLCPCB Part # (none) -> C230306
- R613, R614, R615, R616, R617, R618: JLCPCB Part # (none) -> C17477
- U601, U602: JLCPCB Part # (none) -> C7399456
Changed lines of the file:
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@@
 			)
 		)
-		(property "JLC" ""
+		(property "JLCPCB Part #" "C7399456"
 			(at 104.14 128.27 0)
 			(effects
@@
 			)
 		)
-		(property "JLC" ""
+		(property "JLCPCB Part #" "C473612"
 			(at 41.91 180.34 0)
 			(effects
@@
 			)
 		)
-		(property "Manufacturer_Part_Number" "0402WGF1001TCE"
+		(property "Manufacturer_Part_Number" "FRC0603J103TS"
 			(at 45.72 121.92 0)
 			(effects
@@
 			)
 		)
-		(property "JLC" ""
+		(property "JLCPCB Part #" "C2930027"
 			(at 45.72 121.92 0)
 			(effects
@@
 			)
 		)
-		(property "Value" "20pf"
+		(property "Value" "20p"
 			(at 80.01 176.5299 0)
 			(effects
@@
 			)
 		)
-		(property "JLC" ""
+		(property "JLCPCB Part #" "C1554"
 			(at 76.2 175.26 0)
 			(effects
@@
 			)
 		)
-		(property "JLC" ""
+		(property "JLCPCB Part #" "C473612"
 			(at 41.91 160.02 0)
 			(effects
@@
 			)
 		)
-		(property "Manufacturer_Part_Number" "0402WGF1001TCE"
+		(property "Manufacturer_Part_Number" "FRC0603J103TS"
 			(at 44.45 40.64 0)
 			(effects
@@
 			)
 		)
-		(property "JLC" ""
+		(property "JLCPCB Part #" "C2930027"
 			(at 44.45 40.64 0)
 			(effects
@@
 			)
 		)
-		(property "JLC" ""
+		(property "JLCPCB Part #" "C29266"
 			(at 201.93 80.01 0)
 			(effects
@@
 			)
 		)
-		(property "JLC" ""
+		(property "JLCPCB Part #" "C1525"
 			(at 214.63 80.01 0)
 			(effects
@@
 			)
 		)
-		(property "JLC" ""
+		(property "JLCPCB Part #" "C1525"
 			(at 214.63 52.07 0)
 			(effects
@@
 			)
 		)
-		(property "Value" "20pf"
+		(property "Value" "20p"
 			(at 80.01 166.3699 0)
 			(effects
@@
 			)
 		)
-		(property "JLC" ""
+		(property "JLCPCB Part #" "C1554"
 			(at 76.2 165.1 0)
 			(effects
@@
 			)
 		)
-		(property "JLC" ""
+		(property "JLCPCB Part #" "C7399456"
 			(at 102.87 46.99 0)
 			(effects
@@
 			)
 		)
-		(property "JLC" ""
+		(property "JLCPCB Part #" "C230306"
 			(at 54.61 175.26 0)
 			(effects
@@
 			)
 		)
-		(property "JLC" ""
+		(property "JLCPCB Part #" "C281757"
 			(at 67.31 170.18 0)
 			(effects
@@
 			)
 		)
-		(property "JLC" ""
+		(property "JLCPCB Part #" "C17477"
 			(at 88.9 46.99 0)
 			(effects
@@
 			)
 		)
-		(property "Value" "20pf"
+		(property "Value" "20p"
 			(at 80.01 95.2499 0)
 			(effects
@@
 			)
 		)
-		(property "JLC" ""
+		(property "JLCPCB Part #" "C1554"
 			(at 76.2 93.98 0)
 			(effects
@@
 			)
 		)
-		(property "JLC" ""
+		(property "JLCPCB Part #" "C281757"
 			(at 67.31 88.9 0)
 			(effects
@@
 			)
 		)
-		(property "JLC" ""
+		(property "JLCPCB Part #" "C230306"
 			(at 54.61 83.82 0)
 			(effects
@@
 			)
 		)
-		(property "JLC" ""
+		(property "JLCPCB Part #" "C17477"
 			(at 158.75 137.16 0)
 			(effects
@@
 			)
 		)
-		(property "JLC" ""
+		(property "JLCPCB Part #" "C19702"
 			(at 227.33 80.01 0)
 			(effects
@@
 			)
 		)
-		(property "JLC" ""
+		(property "JLCPCB Part #" "C473612"
 			(at 40.64 78.74 0)
 			(effects
@@
 			)
 		)
-		(property "Value" "20pf"
+		(property "Value" "20p"
 			(at 80.01 85.0899 0)
 			(effects
@@
 			)
 		)
-		(property "JLC" ""
+		(property "JLCPCB Part #" "C1554"
 			(at 76.2 83.82 0)
 			(effects
@@
 			)
 		)
-		(property "JLC" ""
+		(property "JLCPCB Part #" "C29266"
 			(at 227.33 52.07 0)
 			(effects
@@
 			)
 		)
-		(property "JLC" ""
+		(property "JLCPCB Part #" "C17477"
 			(at 88.9 54.61 0)
 			(effects
@@
 			)
 		)
-		(property "JLC" ""
+		(property "JLCPCB Part #" "C230306"
 			(at 54.61 93.98 0)
 			(effects
@@
 			)
 		)
-		(property "Manufacturer_Part_Number" "0402WGF1001TCE"
+		(property "Manufacturer_Part_Number" "FRC0603J103TS"
 			(at 36.83 121.92 0)
 			(effects
@@
 			)
 		)
-		(property "JLC" ""
+		(property "JLCPCB Part #" "C2930027"
 			(at 36.83 121.92 0)
 			(effects
@@
 			)
 		)
-		(property "JLC" ""
+		(property "JLCPCB Part #" "C1554"
 			(at 54.61 142.24 0)
 			(effects
@@
 			)
 		)
-		(property "JLC" ""
+		(property "JLCPCB Part #" "C1525"
 			(at 176.53 50.8 0)
 			(effects
@@
 			)
 		)
-		(property "JLC" ""
+		(property "JLCPCB Part #" "C1554"
 			(at 74.93 60.96 0)
 			(effects
@@
 			)
 		)
-		(property "JLC" ""
+		(property "JLCPCB Part #" "C473612"
 			(at 40.64 99.06 0)
 			(effects
@@
 			)
 		)
-		(property "JLC" ""
+		(property "JLCPCB Part #" "C230306"
 			(at 54.61 165.1 0)
 			(effects
@@
 			)
 		)
-		(property "JLC" ""
+		(property "JLCPCB Part #" "C29266"
 			(at 189.23 50.8 0)
 			(effects
@@
 			)
 		)
-		(property "JLC" ""
+		(property "JLCPCB Part #" "C19702"
 			(at 189.23 80.01 0)
 			(effects
@@
 			)
 		)
-		(property "JLC" ""
+		(property "JLCPCB Part #" "C17477"
 			(at 90.17 135.89 0)
 			(effects
@@
 			)
 		)
-		(property "JLC" ""
+		(property "JLCPCB Part #" "C17477"
 			(at 90.17 128.27 0)
 			(effects
@@
 			)
 		)
-		(property "JLC" ""
+		(property "JLCPCB Part #" "C1525"
 			(at 176.53 80.01 0)
 			(effects
@@
 			)
 		)
-		(property "JLC" ""
+		(property "JLCPCB Part #" "C29266"
 			(at 240.03 80.01 0)
 			(effects
@@
 			)
 		)
-		(property "JLC" ""
+		(property "JLCPCB Part #" "C1554"
 			(at 54.61 60.96 0)
 			(effects
@@
 			)
 		)
-		(property "Manufacturer_Part_Number" "0402WGF1001TCE"
+		(property "Manufacturer_Part_Number" "FRC0603J103TS"
 			(at 35.56 40.64 0)
 			(effects
@@
 			)
 		)
-		(property "JLC" ""
+		(property "JLCPCB Part #" "C2930027"
 			(at 35.56 40.64 0)
 			(effects
@@
 			)
 		)
-		(property "JLC" ""
+		(property "JLCPCB Part #" "C1554"
 			(at 77.47 142.24 0)
 			(effects
@@
 			)
 		)
-		(property "JLC" ""
+		(property "JLCPCB Part #" "C17477"
 			(at 157.48 55.88 0)
 			(effects
