File: MotherBoard/FSAE_BMS.kicad_sch (KiCad schematic)
At the start: 4 parts

Commit message: Daughterboard 100% Complete + Edited Motherboard BOM
Parts:
- H101, H102, H103, H104: now not fitted
Changed lines of the file:
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@@
 		(in_bom no)
 		(on_board yes)
-		(dnp no)
+		(dnp yes)
 		(fields_autoplaced yes)
 		(property "Reference" "H101"
@@
 		(in_bom no)
 		(on_board yes)
-		(dnp no)
+		(dnp yes)
 		(fields_autoplaced yes)
 		(property "Reference" "H102"
@@
 		(in_bom no)
 		(on_board yes)
-		(dnp no)
+		(dnp yes)
 		(fields_autoplaced yes)
 		(property "Reference" "H103"
@@
 		(in_bom no)
 		(on_board yes)
-		(dnp no)
+		(dnp yes)
 		(fields_autoplaced yes)
 		(property "Reference" "H104"
