File: MotherBoard/MCU.kicad_sch (KiCad schematic)
At the start: 42 parts, among them J201 Conn_ARM_SWD_TagConnect_TC2030, J202 DM3AT-SF-PEJM5_40_, U201 STM32F205RBTx, Y201 16 Mhz

Commit message: Daughterboard 100% Complete + Edited Motherboard BOM
Parts:
- J201: now not fitted
- J202: Manufacturer_Part_Number (none) -> DM3AT-SF-PEJM5
Changed lines of the file:
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@@
 		(in_bom no)
 		(on_board yes)
-		(dnp no)
+		(dnp yes)
 		(property "Reference" "J201"
 			(at 60.706 25.4 0)
@@
 			)
 		)
-		(property "Manufacturer_Part_Number" ""
+		(property "Manufacturer_Part_Number" "DM3AT-SF-PEJM5"
 			(at 260.35 830.48 0)
 			(effects

Commit message: Both boards complete
Parts:
- C201, C216: JLCPCB Part # (none) -> C19702
- C202, C205: JLCPCB Part # (none) -> C161520
- C203, C204, C206, C208, C210, C213, C215: JLCPCB Part # (none) -> C1525
- C207, C209: JLCPCB Part # (none) -> C99228
- C211: JLCPCB Part # (none) -> C60133
- C212, C214: JLCPCB Part # (none) -> C29266
- D201, D203, D204, D205, D206, D207, D208, D209: JLCPCB Part # (none) -> C51450
- D202: JLCPCB Part # (none) -> C511604
- J202: JLCPCB Part # (none) -> C114218
- L201: JLCPCB Part # (none) -> C21585
- R201: JLCPCB Part # (none) -> C11702
- R202, R208, R209, R212: JLCPCB Part # (none) -> C2930027; Manufacturer_Part_Number 0402WGF1001TCE -> FRC0603J103TS
- R203: JLCPCB Part # (none) -> C17168
- R204, R205, R206, R207, R210: JLCPCB Part # (none) -> C25092
- R211: JLCPCB Part # (none) -> C25469
- U201: JLCPCB Part # (none) -> C8364
- Y201: JLCPCB Part # (none) -> C13738
Changed lines of the file:
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@@
 			)
 		)
-		(property "JLC" ""
+		(property "JLCPCB Part #" "C51450"
 			(at 69.85 44.45 0)
 			(effects
@@
 			)
 		)
-		(property "JLC" ""
+		(property "JLCPCB Part #" "C25469"
 			(at 217.17 80.01 0)
 			(effects
@@
 			)
 		)
-		(property "JLC" ""
+		(property "JLCPCB Part #" "C51450"
 			(at 36.83 35.56 0)
 			(effects
@@
 			)
 		)
-		(property "JLC" ""
+		(property "JLCPCB Part #" "C25092"
 			(at 124.46 36.83 0)
 			(effects
@@
 			)
 		)
-		(property "JLC" ""
+		(property "JLCPCB Part #" "C19702"
 			(at 234.95 86.36 0)
 			(effects
@@
 			)
 		)
-		(property "JLC" ""
+		(property "JLCPCB Part #" "C8364"
 			(at 99.06 135.89 0)
 			(effects
@@
 			)
 		)
-		(property "JLC" ""
+		(property "JLCPCB Part #" "C17168"
 			(at 59.69 105.41 0)
 			(effects
@@
 			)
 		)
-		(property "JLC" ""
+		(property "JLCPCB Part #" "C60133"
 			(at 119.38 82.55 0)
 			(effects
@@
 			)
 		)
-		(property "JLC" ""
+		(property "JLCPCB Part #" "C29266"
 			(at 130.81 82.55 0)
 			(effects
@@
 			)
 		)
-		(property "JLC" ""
+		(property "JLCPCB Part #" "C161520"
 			(at 46.99 120.65 0)
 			(effects
@@
 			)
 		)
-		(property "Manufacturer_Part_Number" "0402WGF1001TCE"
+		(property "Manufacturer_Part_Number" "FRC0603J103TS"
 			(at 182.88 29.21 0)
 			(effects
@@
 			)
 		)
-		(property "JLC" ""
+		(property "JLCPCB Part #" "C2930027"
 			(at 182.88 29.21 0)
 			(effects
@@
 			)
 		)
-		(property "JLC" ""
-			(at 57.15 34.29 0)
-			(effects
-				(font
-					(size 1.27 1.27)
-				)
-				(hide yes)
-			)
-		)
 		(pin "2"
 		)
@@
 			)
 		)
-		(property "JLC" ""
+		(property "JLCPCB Part #" "C1525"
 			(at 223.52 86.36 0)
 			(effects
@@
 			)
 		)
-		(property "JLC" ""
+		(property "JLCPCB Part #" "C25092"
 			(at 124.46 29.21 0)
 			(effects
@@
 			)
 		)
-		(property "JLC" ""
+		(property "JLCPCB Part #" "C161520"
 			(at 19.05 120.65 0)
 			(effects
@@
 			)
 		)
-		(property "JLC" ""
+		(property "JLCPCB Part #" "C25092"
 			(at 199.39 45.72 0)
 			(effects
@@
 			)
 		)
-		(property "Manufacturer_Part_Number" "0402WGF1001TCE"
+		(property "Manufacturer_Part_Number" "FRC0603J103TS"
 			(at 189.23 29.21 0)
 			(effects
@@
 			)
 		)
-		(property "JLC" ""
+		(property "JLCPCB Part #" "C2930027"
 			(at 189.23 29.21 0)
 			(effects
@@
 			)
 		)
-		(property "JLC" ""
+		(property "JLCPCB Part #" "C511604"
 			(at 39.37 154.94 0)
 			(effects
@@
 			)
 		)
-		(property "Manufacturer_Part_Number" "0402WGF1001TCE"
+		(property "Manufacturer_Part_Number" "FRC0603J103TS"
 			(at 59.69 97.79 0)
 			(effects
@@
 			)
 		)
-		(property "JLC" ""
+		(property "JLCPCB Part #" "C2930027"
 			(at 59.69 97.79 0)
 			(effects
@@
 			)
 		)
-		(property "JLC" ""
+		(property "JLCPCB Part #" "C11702"
 			(at 39.37 163.83 0)
 			(effects
@@
 			)
 		)
-		(property "JLC" ""
+		(property "JLCPCB Part #" "C51450"
 			(at 189.23 59.69 0)
 			(effects
@@
 			)
 		)
-		(property "JLC" ""
+		(property "JLCPCB Part #" "C51450"
 			(at 107.95 44.45 0)
 			(effects
@@
 			)
 		)
-		(property "JLC" ""
+		(property "JLCPCB Part #" "C1525"
 			(at 134.62 44.45 0)
 			(effects
@@
 			)
 		)
-		(property "JLC" ""
+		(property "JLCPCB Part #" "C51450"
 			(at 182.88 59.69 0)
 			(effects
@@
 			)
 		)
-		(property "Manufacturer_Part_Number" "0402WGF1001TCE"
+		(property "Manufacturer_Part_Number" "FRC0603J103TS"
 			(at 275.59 26.67 0)
 			(effects
@@
 			)
 		)
-		(property "JLC" ""
+		(property "JLCPCB Part #" "C2930027"
 			(at 275.59 26.67 0)
 			(effects
@@
 			)
 		)
-		(property "JLC" ""
+		(property "JLCPCB Part #" "C29266"
 			(at 153.67 82.55 0)
 			(effects
@@
 			)
 		)
-		(property "JLC" ""
+		(property "JLCPCB Part #" "C19702"
 			(at 19.05 82.55 0)
 			(effects
@@
 			)
 		)
-		(property "JLC" ""
+		(property "JLCPCB Part #" "C13738"
 			(at 34.29 113.03 0)
 			(effects
@@
 			)
 		)
-		(property "JLC" ""
+		(property "JLCPCB Part #" "C51450"
 			(at 250.19 86.36 0)
 			(effects
@@
 			)
 		)
-		(property "JLC" ""
+		(property "JLCPCB Part #" "C1525"
 			(at 69.85 82.55 0)
 			(effects
@@
 			)
 		)
-		(property "JLC" ""
+		(property "JLCPCB Part #" "C1525"
 			(at 31.75 82.55 0)
 			(effects
@@
 			)
 		)
-		(property "JLC" ""
+		(property "JLCPCB Part #" "C25092"
 			(at 124.46 39.37 0)
 			(effects
@@
 			)
 		)
-		(property "JLC" ""
+		(property "JLCPCB Part #" "C21585"
 			(at 142.24 76.2 0)
 			(effects
@@
 			)
 		)
-		(property "JLC" ""
+		(property "JLCPCB Part #" "C51450"
 			(at 95.25 44.45 0)
 			(effects
@@
 			)
 		)
-		(property "JLC" ""
+		(property "JLCPCB Part #" "C51450"
 			(at 82.55 44.45 0)
 			(effects
@@
 			)
 		)
-		(property "JLC" ""
+		(property "JLCPCB Part #" "C1525"
 			(at 82.55 82.55 0)
 			(effects
@@
 			)
 		)
-		(property "JLC" ""
+		(property "JLCPCB Part #" "C25092"
 			(at 124.46 34.29 0)
 			(effects
@@
 			)
 		)
-		(property "JLC" ""
+		(property "JLCPCB Part #" "C114218"
 			(at 223.52 35.56 0)
 			(effects
@@
 			)
 		)
-		(property "JLC" ""
+		(property "JLCPCB Part #" "C99228"
 			(at 59.69 166.37 0)
 			(effects
@@
 			)
 		)
-		(property "JLC" ""
+		(property "JLCPCB Part #" "C1525"
 			(at 57.15 82.55 0)
 			(effects
@@
 			)
 		)
-		(property "JLC" ""
+		(property "JLCPCB Part #" "C1525"
 			(at 44.45 82.55 0)
 			(effects
@@
 			)
 		)
-		(property "JLC" ""
+		(property "JLCPCB Part #" "C99228"
 			(at 72.39 166.37 0)
 			(effects
